File: hardware/d1/DrunkEarPhoneAdapter.kicad_pcb (KiCad board)
At the start: 4 copper layers, 40.3 x 34.7 mm, 144 parts, among them Q1 CSD17577Q3A, Q2 CSD17577Q3A, SW1 SSSS811101, U1 CS43131-CNZR, U10 BLM15PX601SN1D, U11 TPS7A2033PDBVR, U12 TPS7A2018PDBVR, U13 TPS7A2018PDBVR, U14 BLM15PX601SN1D, U15 ESDA25P35-1U1M, U16 ESDA25P35-1U1M, U18 TPS22917DBVR, U19 TPS22917DBVR, U2 STM32G0B1VCT6, U4 TCPP03-M20, U5 TCPP03-M20, U6 ES8327, U7 TPS7A2018PDBVR, U8 TPS7A2033PDBVR, U9 TPS560430XFDBVR, X1 22.5792MHz, X3 24.576MHz

Commit message: Fixes
Parts:
- removed C69, C75: 100nF 50V X7R, JLCImport:CL05B104KB54PNC
- removed C9: 1uF 25V X5R, JLCImport:CL05A105KA5NQNC
- removed R1, R7: 33Ω, Resistor_SMD:R_0402_1005Metric
- added C80: 1nF 50V X7R, Capacitor_SMD:C_0402_1005Metric, F.Cu at (94.2, 16.2)
- added C81: 1nF 50V X7R, Capacitor_SMD:C_0402_1005Metric, F.Cu at (94.2, 18.2)
- added C82: 1nF 50V X7R, Capacitor_SMD:C_0402_1005Metric, F.Cu at (94.2, 20.1)
- added C83: 1nF 50V X7R, Capacitor_SMD:C_0402_1005Metric, F.Cu at (94.2, 22.1)
- added C84: 22uF 25V X5R, JLCImport:CL21A226MAQNNNE, F.Cu at (68.3, 58.8)
- added C85: 22uF 25V X5R, JLCImport:CL21A226MAQNNNE, F.Cu at (68.3, 61.7)
- added C86: 100nF 50V X7R, Capacitor_SMD:C_0402_1005Metric, F.Cu at (106.1, 102.5)
- added C87: 100nF 50V X7R, Capacitor_SMD:C_0402_1005Metric, F.Cu at (113.3, 106.5)
- added C88: 100nF 50V X7R, Capacitor_SMD:C_0402_1005Metric, F.Cu at (113.3, 108.5)
- added D4: TPD4E1B06DCKR, JLCImport:TPD4E1B06DCKR, F.Cu at (74.9, 59.0)
- added R31: 100kΩ, JLCImport:0402WGF1003TCE, F.Cu at (89.2, 16.3)
- added R32: 100kΩ, JLCImport:0402WGF1003TCE, F.Cu at (89.2, 18.4)
- added R33: 100kΩ, JLCImport:0402WGF1003TCE, F.Cu at (89.2, 20.6)
- added R34: 100kΩ, JLCImport:0402WGF1003TCE, F.Cu at (89.2, 22.7)
- added R35: 1kΩ, Resistor_SMD:R_0402_1005Metric, F.Cu at (113.2, 99.6)
- added U17: SN74LVC1G32DBVR, Package_TO_SOT_SMD:SOT-23-5, F.Cu at (107.3, 107.9)
- C4: value 100nF 50V X7R -> 2.2uF 50V X7R; footprint JLCImport:CL05B104KB54PNC -> JLCImport:CC0805KKX7R9BB225
- D1, D3: footprint Diode_SMD:D_SOD-110 -> Diode_SMD:D_SOD-123F
- D2: value B5819WS_C916992 -> PMEG4010CEH_115; footprint Diode_SMD:D_SOD-323 -> Diode_SMD:D_SOD-123F
- moved C4 76.8 mm to (107.2, 100.1)
- moved D3 50.5 mm to (49.4, 24.1)
- moved D1 43.3 mm to (55.9, 24.6)
- moved USBC2 23.2 mm to (38.7, 46.7)
- moved D2 17.2 mm to (77.8, 23.0)
- moved U6 16.6 mm to (46.8, 31.9)
Connections:
- Audio1 pad 4: +3V3_D -> GND
- Audio1 pad 6: +3V3_D -> GND
- Audio1 pad 7: +3V3_D -> GND
- C10 pad 1: +3V3_D -> GND
- C11 pad 1: +3V3_D -> GND
- C12 pad 1: +3V3_D -> GND
- C13 pad 1: +3V3_D -> GND
- C14 pad 1: +3V3_D -> GND
- C15 pad 1: +3V3_D -> GND
- C16 pad 2: +3V3_D -> GND
- C17 pad 1: +3V3_D -> GND
- C18 pad 2: +3V3_D -> GND
- C19 pad 2: +3V3_D -> GND
- C2 pad 2: +3V3_D -> GND
- C20 pad 2: +3V3_D -> GND
- C21 pad 1: +3V3_D -> GND
- C22 pad 2: +3V3_D -> GND
- C23 pad 1: +3V3_D -> GND
- C24 pad 2: +3V3_D -> GND
- C25 pad 2: +3V3_D -> GND
- C28 pad 2: +3V3_D -> GND
- C3 pad 2: +3V3_D -> GND
- C30 pad 2: +3V3_D -> GND
- C31 pad 2: +3V3_D -> GND
- C32 pad 1: +3V3_D -> GND
- C35 pad 2: +3V3_D -> GND
- C36 pad 2: +3V3_D -> GND
- C37 pad 2: +3V3_D -> GND
- C38 pad 2: +3V3_D -> GND
- C39 pad 2: +3V3_D -> GND
- C4 pad 1: PWR_IN -> +3V3_A
- C4 pad 2: +3V3_D -> GND
- C40 pad 2: +3V3_D -> GND
- C41 pad 2: +3V3_D -> GND
- C42 pad 2: +3V3_D -> GND
- C43 pad 2: +3V3_D -> GND
- C44 pad 2: +3V3_D -> GND
- C45 pad 2: +3V3_D -> GND
- C47 pad 2: +3V3_D -> GND
- C49 pad 1: +3V3_D -> GND
- C49 pad 2: /mcu/ADC1_IN5 -> /mcu/ADC1_IN4
- C5 pad 2: +3V3_D -> GND
- C50 pad 2: +3V3_D -> GND
- C51 pad 1: +3V3_D -> GND
- C52 pad 2: +3V3_D -> GND
- C53 pad 2: +3V3_D -> GND
- C54 pad 2: +3V3_D -> GND
- C55 pad 2: +3V3_D -> GND
- C56 pad 2: +3V3_D -> GND
- C57 pad 1: +3V3_D -> GND
- C58 pad 1: +3V3_D -> GND
- C59 pad 1: +3V3_D -> GND
- C6 pad 1: +3V3_D -> GND
- C60 pad 1: +3V3_D -> GND
- C61 pad 1: +3V3_D -> GND
- C62 pad 1: +3V3_D -> GND
- C63 pad 1: +3V3_D -> GND
- C64 pad 1: +3V3_D -> GND
- C67 pad 2: +3V3_D -> GND
- C68 pad 2: +3V3_D -> GND
- C7 pad 1: +3V3_D -> GND
- C70 pad 1: +3V3_D -> GND
- C71 pad 1: +3V3_D -> GND
- C72 pad 1: +3V3_D -> GND
- C73 pad 1: +3V3_D -> GND
- C74 pad 2: +3V3_D -> GND
- C76 pad 1: +3V3_D -> GND
- C77 pad 2: +3V3_D -> GND
- C78 pad 2: +3V3_D -> GND
- C79 pad 2: +3V3_D -> GND
- C8 pad 1: +3V3_D -> GND
- L7 pad 3: +3V3_D -> GND
- R11 pad 2: /mcu/I2C2_SCL -> /adc/I2C_SCL
- R12 pad 2: /mcu/I2C2_SDA -> /adc/I2C_SDA
- R14 pad 1: /mcu/ADC1_IN5 -> /mcu/ADC1_IN4
- R15 pad 1: +3V3_D -> GND
- R15 pad 2: /mcu/ADC1_IN5 -> /mcu/ADC1_IN4
- R20 pad 1: +3V3_D -> GND
- R22 pad 1: +3V3_D -> GND
- R23 pad 1: /mcu/ADC1_IN2 -> /mcu/ADC1_IN0
- R24 pad 1: /mcu/GPIO_EXTI3 -> /mcu/GPIO_EXTI2
- R25 pad 1: /mcu/GPIO_EXTI4 -> /mcu/GPIO_EXTI3
- R27 pad 1: +3V3_D -> GND
- R29 pad 1: +3V3_D -> GND
- R3 pad 2: +3V3_D -> GND
- R30 pad 1: /mcu/ADC1_IN4 -> /mcu/ADC1_IN2
- R4 pad 1: /dac/DAC_RESET -> /dac/DAC_RESET/
- R5 pad 1: +3V3_D -> GND
- R8 pad 1: +3V3_D -> GND
- SW1 pad 1: +3V3_D -> GND
- SW1 pad 2: +3V3_D -> GND
- SW1 pad 4: +3V3_D -> GND
- SW1 pad 5: +3V3_D -> GND
- SW1 pad 6: +3V3_D -> GND
- SW1 pad 7: +3V3_D -> GND
- U1 pad 13: +3V3_D -> GND
- U1 pad 17: +3V3_D -> GND
- U1 pad 19: +3V3_D -> GND
- U1 pad 28: /dac/DAC_RESET -> /dac/DAC_RESET/
- U1 pad 30: +3V3_D -> GND
- U1 pad 35: +3V3_D -> GND
- U1 pad 36: +3V3_D -> GND
- U1 pad 41: +3V3_D -> GND
- U1 pad 8: +3V3_D -> GND
- U11 pad 2: +3V3_D -> GND
- U12 pad 2: +3V3_D -> GND
- U13 pad 2: +3V3_D -> GND
- U15 pad 2: +3V3_D -> GND
- U16 pad 2: +3V3_D -> GND
- U18 pad 2: +3V3_D -> GND
- U19 pad 2: +3V3_D -> GND
- U2 pad 14: +3V3_D -> GND
- U2 pad 25: /mcu/ADC1_IN1 -> /mcu/ADC1_IN0
- U2 pad 26: /mcu/ADC1_IN2 -> /mcu/ADC1_IN1
- U2 pad 27: /mcu/ADC1_IN3 -> /mcu/ADC1_IN2
- U2 pad 28: /mcu/ADC1_IN4 -> /mcu/ADC1_IN3
- U2 pad 29: /mcu/ADC1_IN5 -> /mcu/ADC1_IN4
- U2 pad 56: unconnected-(U2-PA9-Pad56) -> /mcu/UCPD1_DBCC1
- U2 pad 63: +3V3_D -> GND
- U2 pad 69: unconnected-(U2-PA10-Pad69) -> /mcu/UCPD1_DBCC2
- U2 pad 79: unconnected-(U2-PD1-Pad79) -> /mcu/UCPD2_DBCC1
- U2 pad 81: unconnected-(U2-PD3-Pad81) -> /mcu/UCPD2_DBCC2
- U2 pad 83: unconnected-(U2-PD5-Pad83) -> /dac/CLOCK_EN_24_576
- U2 pad 84: unconnected-(U2-PD6-Pad84) -> /dac/CLOCK_EN_22_5792
- U2 pad 85: unconnected-(U2-PD7-Pad85) -> /dac/DAC_RESET/
- U2 pad 94: unconnected-(U2-PE0-Pad94) -> /dac//INT
- U2 pad 95: unconnected-(U2-PE1-Pad95) -> /adc/INT/
- U2 pad 96: unconnected-(U2-PE2-Pad96) -> /mcu/GPIO_EXTI2
- U2 pad 97: unconnected-(U2-PE3-Pad97) -> /mcu/GPIO_EXTI3
- U2 pad 98: /mcu/I2C2_SCL -> /adc/I2C_SCL
- U2 pad 99: /mcu/I2C2_SDA -> /adc/I2C_SDA
- U4 pad 12: +3V3_D -> GND
- U4 pad 16: +3V3_D -> GND
- U4 pad 19: /mcu/GPIO_EXTI3 -> /mcu/GPIO_EXTI2
- U4 pad 21: +3V3_D -> GND
- U5 pad 12: +3V3_D -> GND
- U5 pad 19: /mcu/GPIO_EXTI4 -> /mcu/GPIO_EXTI3
- U5 pad 21: +3V3_D -> GND
- U6 pad 13: +3V3_D -> GND
- U6 pad 14: +3V3_D -> GND
- U6 pad 22: +3V3_D -> GND
- U6 pad 30: +3V3_D -> GND
- U6 pad 33: +3V3_D -> GND
- U6 pad 4: +3V3_D -> GND
- U6 pad 6: +3V3_D -> GND
- U7 pad 2: +3V3_D -> GND
- U8 pad 2: +3V3_D -> GND
- U9 pad 2: +3V3_D -> GND
- USBC1 pad 0: +3V3_D -> GND
- USBC1 pad A1: +3V3_D -> GND
- USBC1 pad A12: +3V3_D -> GND
- USBC1 pad B1: +3V3_D -> GND
- USBC1 pad B12: +3V3_D -> GND
- USBC2 pad 5: +3V3_D -> GND
- X1 pad 2: +3V3_D -> GND
- X3 pad 2: +3V3_D -> GND

Commit message: Fixes
Parts:
- removed R16: 33Ω 0805, Resistor_SMD:R_0805_2012Metric
- removed R8: 10kΩ, Resistor_SMD:R_0402_1005Metric
- removed SW1: SSSS811101, JLCImport:SSSS811101
- added C89: 100nF 16V X7R, JLCImport:CL05B104KO5NNNC, F.Cu at (99.1, 116.0)
- added C90: 100nF 16V X7R, JLCImport:CL05B104KO5NNNC, F.Cu at (99.1, 118.1)
- added C91: 100nF 16V X7R, JLCImport:CL05B104KO5NNNC, F.Cu at (99.1, 120.3)
- added C92: 100nF 16V X7R, JLCImport:CL05B104KO5NNNC, F.Cu at (99.1, 122.4)
- added R1: 100Ω 1206, Resistor_SMD:R_1206_3216Metric, F.Cu at (75.9, 36.4)
- added R36: 100kΩ, JLCImport:0402WGF1003TCE, F.Cu at (99.2, 128.4)
- added R7: 100kΩ, JLCImport:0402WGF1003TCE, F.Cu at (102.1, 120.3)
- added SW2: DSHP04TS-S, JLCImport:DSHP04TS-S, F.Cu at (45.5, 41.0)
- added TP1: 3V3_D, TestPoint:TestPoint_Pad_1.0x1.0mm, F.Cu at (68.5, 36.2)
- added TP2: 1V8_D, TestPoint:TestPoint_Pad_1.0x1.0mm, F.Cu at (68.5, 39.3)
- added TP3: 1V8_CP, TestPoint:TestPoint_Pad_1.0x1.0mm, F.Cu at (68.5, 42.3)
- added TP4: 1V8_VA, TestPoint:TestPoint_Pad_1.0x1.0mm, F.Cu at (68.5, 45.4)
- added TP5: 3V3_VA, TestPoint:TestPoint_Pad_1.0x1.0mm, F.Cu at (71.6, 36.2)
- added TP6: 3V8, TestPoint:TestPoint_Pad_1.0x1.0mm, F.Cu at (71.6, 39.3)
- added TP7: PWR_IN, TestPoint:TestPoint_Pad_1.0x1.0mm, F.Cu at (71.6, 42.3)
- added U20: SN74AVC4T774RSVR, JLCImport:SN74AVC4T774RSVR, F.Cu at (105.7, 121.3)
- added U21: TCA9406DCUR, JLCImport:TCA9406DCUR, F.Cu at (105.6, 117.3)
- R5: value 10kΩ -> 100kΩ; footprint Resistor_SMD:R_0402_1005Metric -> JLCImport:0402WGF1003TCE
- moved R9 64.8 mm to (102.0, 122.3)
- moved R4 46.1 mm to (102.1, 116.0)
- moved R35 27.1 mm to (102.0, 124.3)
- moved R5 15.1 mm to (102.1, 118.1)
Connections:
- C18 pad 1: Net-(U2-VREF+) -> Net-(U2-VBAT)
- C20 pad 1: Net-(U2-VREF+) -> Net-(U2-VBAT)
- C40 pad 1: +1V8_D -> +3V3_D
- C50 pad 1: +1V8_D -> +3V3_D
- C52 pad 1: +1V8_D -> Net-(U2-VBAT)
- C53 pad 1: +1V8_D -> +3V3_D
- C56 pad 1: Net-(U2-PF2-NRST) -> GND
- C56 pad 2: GND -> /mcu/NRST
- D4 pad 4: Net-(D4-IO3) -> /dac/JACK_TIP_DETECT
- L4 pad 1: +1V8_D -> +3V3_D
- L4 pad 2: Net-(U2-VREF+) -> Net-(U2-VBAT)
- R10 pad 2: +1V8_D -> +3V3_D
- R11 pad 1: +1V8_D -> +3V3_D
- R12 pad 1: +1V8_D -> +3V3_D
- R13 pad 2: +1V8_D -> +3V3_D
- R24 pad 2: +1V8_D -> +3V3_D
- R25 pad 2: +1V8_D -> +3V3_D
- R35 pad 1: Net-(D4-IO3) -> Net-(U1-HP_DETECT)
- R4 pad 1: /dac/DAC_RESET/ -> GND
- R4 pad 2: +1V8_D -> /dac/DAC_RESET/
- R6 pad 2: +1V8_D -> +3V3_D
- R9 pad 1: Net-(U1-CLKOUT) -> Net-(U20-B3)
- U1 pad 1: /adc/I2C_SCL -> /dac/I2C_SCL_1v8
- U1 pad 2: /dac/I2S_SD -> /dac/I2S_SD_1v8
- U1 pad 22: /dac/JACK_TIP_DETECT -> Net-(U1-HP_DETECT)
- U1 pad 33: Net-(U1-CLKOUT) -> /dac/CLKOUT_1v8
- U1 pad 34: /dac/I2S_CK -> /dac/I2S_CK_1v8
- U1 pad 38: /dac/I2S_WS -> /dac/I2S_WS_1v8
- U1 pad 39: /adc/I2C_SDA -> /dac/I2C_SDA_1v8
- U2 pad 11: +1V8_D -> Net-(U2-VBAT)
- U2 pad 12: Net-(U2-VREF+) -> Net-(U2-VBAT)
- U2 pad 13: +1V8_D -> +3V3_D
- U2 pad 17: Net-(U2-PF2-NRST) -> /mcu/NRST
- U2 pad 86: unconnected-(U2-PF9-Pad86) -> /mcu/PHONE_EN
- U4 pad 20: +1V8_D -> /mcu/PHONE_EN
- U5 pad 16: +1V8_D -> +3V3_D
- U5 pad 20: +1V8_D -> +3V3_D
- U6 pad 3: +1V8_D -> +3V3_D
- U8 pad 3: +1V8_D -> +3V8

Commit message: Fixesss
Parts:
- added J3: SWD, JLCImport:Conn_1x5_1.27, F.Cu at (37.8, 17.3)
- added J4: UART, JLCImport:Conn_1x5_1.27, F.Cu at (37.8, 19.3)
- moved SW2 21.5 mm to (63.2, 28.9)
- moved Audio1 7.24 mm to (60.3, 44.3)
- moved USBC2 6.75 mm to (45.4, 45.9)
- moved USBC1 2.74 mm to (29.9, 50.9)
Connections:
- C65 pad 1: unconnected-(C65-Pad1) -> GND
Other:
- board size 40.3 x 34.7 mm -> 50 x 35 mm

Commit message: Fixes
Parts:
- removed C2, C3: 2.2uF 50V X7R, JLCImport:CC0805KKX7R9BB225
- removed C85: 22uF 25V X5R, JLCImport:CL21A226MAQNNNE
- removed R26: 10kΩ, Resistor_SMD:R_0402_1005Metric
- removed R27: 560Ω, Resistor_SMD:R_0402_1005Metric
- added C69: 100nF 16V X7R, JLCImport:CL05B104KO5NNNC, F.Cu at (136.8, 45.4)
- added C75: 22uF 25V X5R, JLCImport:CL21A226MAQNNNE, F.Cu at (127.7, 23.7)
- added C9: 47uF 25V X5R, Capacitor_SMD:C_1206_3216Metric, F.Cu at (55.0, 60.5)
- added C93: 1uF 25V X5R, JLCImport:CL05A105KA5NQNC, F.Cu at (133.7, 23.3)
- added C94: 1uF 25V X5R, JLCImport:CL05A105KA5NQNC, F.Cu at (133.7, 25.4)
- added L8: ECMF02-2AMX6, JLCImport:ECMF02-2AMX6, F.Cu at (22.5, 82.3)
- added NT1: NetTie_2, NetTie:NetTie-2_SMD_Pad0.5mm, F.Cu at (89.0, 42.9)
- added NT2: NetTie_3, NetTie:NetTie-3_SMD_Pad0.5mm, F.Cu at (89.5, 41.4)
- added Q3: DMG1012T-7, Package_TO_SOT_SMD:SOT-523, F.Cu at (134.2, 42.7)
- added R16: 33Ω, Resistor_SMD:R_0402_1005Metric, F.Cu at (136.6, 27.5)
- added R37: 100kΩ, JLCImport:0402WGF1003TCE, F.Cu at (136.7, 25.4)
- added R38: 33Ω, Resistor_SMD:R_0402_1005Metric, F.Cu at (136.6, 29.5)
- added R39: 100kΩ, JLCImport:0402WGF1003TCE, F.Cu at (133.8, 45.4)
- added R40: 10kΩ 0603, Resistor_SMD:R_0603_1608Metric, F.Cu at (86.0, 29.9)
- added R41: 10kΩ 0603, Resistor_SMD:R_0603_1608Metric, F.Cu at (86.0, 32.4)
- added R42: 100kΩ, JLCImport:0402WGF1003TCE, F.Cu at (23.0, 76.8)
- added R8: 100kΩ, JLCImport:0402WGF1003TCE, F.Cu at (136.7, 23.3)
- added SW1: SSSS811101, JLCImport:SSSS811101, F.Cu at (45.2, 53.5)
- added U3: TS3USB221RSER, JLCImport:TS3USB221RSER, F.Cu at (19.2, 82.2)
- C51, C57, C58, C59, C60, C61, C62, C63: value 22uF 25V X5R -> 47uF 25V X5R; footprint JLCImport:CL21A226MAQNNNE -> Capacitor_SMD:C_1206_3216Metric
- C64, C65: value 22uF 25V X5R -> 2.2uF 50V X7R; footprint JLCImport:CL21A226MAQNNNE -> Capacitor_SMD:C_1206_3216Metric
- C67, C68: footprint JLCImport:CC0805KKX7R9BB225 -> Capacitor_SMD:C_1206_3216Metric
- C84: value 22uF 25V X5R -> 100nF 16V X7R; footprint JLCImport:CL21A226MAQNNNE -> JLCImport:CL05B104KO5NNNC
- R19: value 10kΩ -> 510Ω; footprint Resistor_SMD:R_0402_1005Metric -> Resistor_SMD:R_0603_1608Metric
- R20: value 560Ω -> 510Ω; footprint Resistor_SMD:R_0402_1005Metric -> Resistor_SMD:R_0603_1608Metric
- moved C68 118.9 mm to (122.4, 37.3)
- moved C67 118.8 mm to (122.4, 33.9)
- moved R20 65.1 mm to (19.5, 79.5)
- moved R19 64.6 mm to (19.5, 77.0)
- moved C64 52.8 mm to (135.1, 34.1)
- moved C65 52.6 mm to (135.1, 37.5)
- moved C84 49.7 mm to (23.0, 79.0)
- moved C60 46.7 mm to (55.0, 77.2)
- moved C59 46.4 mm to (55.0, 73.9)
- moved C58 46.1 mm to (55.0, 70.5)
- moved C57 45.9 mm to (55.0, 67.2)
- moved C51 45.6 mm to (55.0, 63.9)
- moved C61 42.0 mm to (122.4, 23.9)
- moved C62 41.8 mm to (122.4, 27.2)
- moved C63 41.6 mm to (122.4, 30.6)
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Connections:
- C18 pad 1: Net-(U2-VBAT) -> Net-(U2-VREF+)
- C20 pad 1: Net-(U2-VBAT) -> Net-(U2-VREF+)
- C47 pad 2: GND -> /adc/GMS0
- C52 pad 1: Net-(U2-VBAT) -> Net-(U2-VREF+)
- C64 pad 2: Net-(D2-A) -> /ucpd/USB_PHONE_VBUS
- C65 pad 2: Net-(D2-A) -> /ucpd/USB_CHR_VBUS
- C67 pad 1: /ucpd/USB_CHR_VBUS -> GND
- C67 pad 2: GND -> PWR_IN
- C68 pad 1: /ucpd/USB_PHONE_VBUS -> GND
- C68 pad 2: GND -> PWR_IN
- C84 pad 1: GND -> +3V3_D
- C84 pad 2: Net-(D2-A) -> GND
- L4 pad 2: Net-(U2-VBAT) -> Net-(U2-VREF+)
- L7 pad 1: /mcu/USB_DP -> /ucpd/USB_PHONE_SAFE_DP
- L7 pad 2: /mcu/USB_DN -> /ucpd/USB_PHONE_SAFE_DN
- R19 pad 1: /ucpd/VSENSE_PHONE -> GND
- R19 pad 2: /ucpd/USB_PHONE_VBUS -> /ucpd/VSENSE_PHONE
- R20 pad 2: /ucpd/VSENSE_PHONE -> /ucpd/VSENSE_CHR
- U1 pad 13: GND -> /dac/HPREFA
- U1 pad 17: GND -> /dac/HPREFB
- U17 pad 4: Net-(U1-XTI/MCLK) -> Net-(U17-Y)
- U2 pad 11: Net-(U2-VBAT) -> +3V3_D
- U2 pad 12: Net-(U2-VBAT) -> Net-(U2-VREF+)
- U2 pad 51: unconnected-(U2-PB12-Pad51) -> /mcu/UCPD2_FRSTX1
- U2 pad 53: unconnected-(U2-PB14-Pad53) -> /mcu/UCPD1_FRSTX2
- U2 pad 59: unconnected-(U2-PD8-Pad59) -> /mcu/USB_DIR
- U2 pad 60: unconnected-(U2-PD9-Pad60) -> /mcu/USB_DIR_SW
- U2 pad 7: unconnected-(U2-PC12-Pad7) -> /mcu/UCPD1_FRSTX1
- U2 pad 76: unconnected-(U2-PC8-Pad76) -> /mcu/UCPD2_FRSTX2
- U20 pad 12: /dac/I2S_CK -> Net-(U20-B1)
- U6 pad 13: GND -> /adc/GMS0
Other:
- outline, holes or cut-outs redrawn
