File: hardware/d1/DrunkEarPhoneAdapter.kicad_pcb (KiCad board)
At the start: 4 copper layers, 50 x 50 mm, 191 parts, among them J3 SWD, J4 UART, Q1 CSD17577Q3A, Q2 CSD17577Q3A, Q3 DMG1012T-7, SW1 SSSS811101, SW2 DSHP04TS-S, U1 CS43131-CNZR, U10 BLM15PX601SN1D, U11 TPS7A2033PDBVR, U12 TPS7A2018PDBVR, U13 TPS7A2018PDBVR, U14 BLM15PX601SN1D, U15 ESDA25P35-1U1M, U16 ESDA25P35-1U1M, U17 SN74LVC1G32DBVR, U18 TPS22917DBVR, U19 TPS22917DBVR, U2 STM32G0B1VCT6, U20 SN74AVC4T774RSVR, U21 TCA9406DCUR, U3 TS3USB221RSER, U4 TCPP03-M20, U5 TCPP03-M20, U6 ES8327, U7 TPS7A2018PDBVR, U8 TPS7A2033PDBVR, U9 TPS560430XFDBVR, X1 22.5792MHz, X3 24.576MHz

Commit message: Almost done tracing
Parts:
- removed C33: 330pF 50V, Capacitor_SMD:C_0603_1608Metric
- removed C63: 47uF 25V X5R, Capacitor_SMD:C_1206_3216Metric
- removed C66: 10nF 50V X7R, Capacitor_SMD:C_0402_1005Metric
- removed JP2, JP3, JP4: SolderJumper_2_Bridged, Jumper:SolderJumper-2_P1.3mm_Bridged_RoundedPad1.0x1.5mm
- removed SW2: DSHP04TS-S, JLCImport:DSHP04TS-S
- added SW3: DSHP02TSGER, JLCImport:DSHP02TSGER, F.Cu at (47.6, 43.4)
- C17, C19, C22, C28, C30, C39, C49, C56, C65, C76, C77, C78, C91, C92, C98, J3, J4, R11, R12, R14, R15, R24, R25, R26, R28, R29, R35, R38, R5, R7, R9, U20: moved to B.Cu
- moved R1 275.7 mm to (22.5, 27.9), turned to -90 degrees
- moved D2 269.6 mm to (25.0, 27.9), turned to -90 degrees
- moved C60 261.1 mm to (22.1, 52.3)
- moved C59 260.8 mm to (22.1, 49.8)
- moved C58 260.5 mm to (22.1, 47.2)
- moved C57 260.2 mm to (22.1, 44.7)
- moved C51 260.0 mm to (22.1, 42.1)
- moved C9 259.7 mm to (22.1, 39.6)
- moved C62 257.9 mm to (22.1, 37.1)
- moved C61 257.7 mm to (22.1, 34.6)
- moved C106 130.6 mm to (30.8, 34.8)
- moved C56 130.4 mm to (40.6, 26.2), turned to 90 degrees
- moved C39 129.0 mm to (61.3, 28.9), turned to 90 degrees
- moved C100 122.5 mm to (30.4, 41.0), turned to 180 degrees
- moved C37 122.3 mm to (28.2, 34.5)
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Connections:
- U2 pad 51: /mcu/UCPD2_FRSTX1 -> unconnected-(U2-PB12-Pad51)
- U2 pad 53: /mcu/UCPD1_FRSTX2 -> unconnected-(U2-PB14-Pad53)
- U2 pad 76: /mcu/UCPD2_FRSTX2 -> unconnected-(U2-PC8-Pad76)
- U4 pad 13: /ucpd/USB_PHONE_CC2 -> unconnected-(U4-CC2c-Pad13)
- U4 pad 8: /ucpd/GDCs -> unconnected-(U4-GDCs-Pad8)
- U5 pad 6: /ucpd/GDPs_CHR -> unconnected-(U5-GDPs-Pad6)
- U5 pad 8: /ucpd/GDCs_CHR -> unconnected-(U5-GDCs-Pad8)
Routing:
- net /adc/I2C_SCL: track 0.00 -> 80.1 mm, vias 0 -> 11
- net /adc/I2S_CK: track 0.00 -> 77.1 mm, vias 0 -> 3
- net /adc/I2C_SDA: track 0.00 -> 75.9 mm, vias 0 -> 8
- net GND: track 55.2 -> 117.8 mm, vias 218 -> 271
- net /adc/I2S_SD: track 0.00 -> 51.0 mm, vias 0 -> 3
- net /dac/DAC_RESET/: track 3.46 -> 40.7 mm, vias 0 -> 3
- net /mcu/ADC1_IN0: track 0.00 -> 36.7 mm, vias 0 -> 2
- net /mcu/UCPD2_CC1: track 0.00 -> 34.1 mm, vias 0 -> 5
- net /adc/GMS0: track 29.9 -> 62.6 mm, vias 1 -> 0
- net /adc/INT/: track 7.67 -> 39.9 mm, vias 0 -> 3
- net /dac/I2S_WS: track 0.00 -> 30.4 mm, vias 0 -> 2
- net /dac/I2S_SD: track 0.00 -> 30.2 mm, vias 0 -> 2
- net /mcu/UCPD2_CC2: track 0.00 -> 29.6 mm, vias 0 -> 3
- net /mcu/UCPD1_FRSTX1: track 0.00 -> 27.7 mm, vias 0 -> 3
- net /adc/GMS1: track 29.7 -> 56.1 mm, vias 3 -> 5
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Other:
- board text added: "+3v3"
- board text added: "Drunk"
- board text added: "GND"
- board text added: "Head"
- board text added: "SWCLK"
- board text added: "SWD"
- board text added: "SWDIO"
- board text added: "UART"
