File: hardware/d1/DrunkEarPhoneAdapter.kicad_sch (KiCad schematic)
At the start: 0 parts

Commit message: Pre-finalize sch
Other:
- sheet adc ports: added CLKIN, I2C_SCL, I2C_SDA, I2S_CK, I2S_SD, I2S_WS, INT/, JACK_RING_2, JACK_SLEEVE; removed none
- sheet dac ports: added CLKOUT, CLOCK_EN_22_5792, CLOCK_EN_24_576, I2C_SCL, I2C_SDA, I2S_CK, I2S_SD, I2S_WS, JACK_RING_1, JACK_RING_2, JACK_TIP, JACK_TIP_DETECT, /INT; removed none
- sheet headset ports: added JACK_RING_1, JACK_RING_2, JACK_SLEEVE, JACK_TIP, JACK_TIP_DETECT; removed none
- sheet mcu ports: added ADC1_IN1, ADC1_IN2, ADC1_IN3, ADC1_IN4, CLOCK_EN_22_5792, CLOCK_EN_24_576, GPIO_EXTI1, GPIO_EXTI2, GPIO_EXTI3, GPIO_EXTI4, I2C1_SCL, I2C1_SDA, I2S1_CK, I2S1_SD, I2S1_WS, I2S2_CK, I2S2_SD, I2S2_WS, JACK_SLEEVE, UCPD1_CC1, UCPD1_CC2, UCPD2_CC1, UCPD2_CC2, USB_DN, USB_DP; removed none
- sheet ucpd ports: added ADC_CHR_IANA, ADC_CHR_VBUS, ADC_PHONE_IANA, ADC_PHONE_VBUS, CHR_INT/, I2C1_SCL, I2C1_SDA, PHONE_INT/, UCPD1_CC1, UCPD1_CC2, UCPD2_CC1, UCPD2_CC2, USB_DN, USB_DP; removed none

Commit message: Fixes
Other:
- sheet dac ports: added DAC_RESET/; removed none
- sheet mcu ports: added ADC1_IN0, CS_RESET/, GPIO_EXTI0; removed ADC1_IN4, GPIO_EXTI4

Commit message: Fixes
Other:
- sheet mcu ports: added PHONE_EN; removed none
- sheet ucpd ports: added PHONE_EN; removed none
Changed lines of the file:
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@@
+	(wire
+		(pts
+			(xy 78.74 135.89) (xy 218.44 135.89)
+		)
+		(stroke
+			(width 0)
+			(type default)
+		)
+	)
 	(wire
 		(pts
@@
 		(pts
 			(xy 78.74 87.63) (xy 189.23 87.63)
+		)
+		(stroke
+			(width 0)
+			(type default)
+		)
+	)
+	(wire
+		(pts
+			(xy 218.44 135.89) (xy 218.44 140.97)
 		)
 		(stroke
@@
 			)
 		)
+		(pin "PHONE_EN" input
+			(at 218.44 140.97 90)
+			(effects
+				(font
+					(size 1.27 1.27)
+				)
+				(justify right)
+			)
+		)
 		(instances
 			(project "DrunkEarPhoneAdapter"
@@
 			(effects
 				(font
+					(size 1.27 1.27)
+				)
+				(justify right)
+			)
+		)
+		(pin "PHONE_EN" output
+			(at 78.74 135.89 0)
+			(effects
+				(font

Commit message: Fixes
Other:
- sheet adc ports: added HP_GND; removed JACK_RING_2
- sheet dac ports: added HPREFA, HPREFB; removed JACK_RING_2
- sheet headset ports: added ES_GND, HPREFA, HPREFB; removed JACK_RING_2
- sheet ucpd ports: added USB_DIR; removed none

Commit message: Fixes
Other:
- sheet mcu ports: added USB_DIR; removed none
Changed lines of the file:
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@@
+	(wire
+		(pts
+			(xy 255.27 182.88) (xy 255.27 196.85)
+		)
+		(stroke
+			(width 0)
+			(type default)
+		)
+	)
 	(wire
 		(pts
@@
 		(pts
 			(xy 246.38 168.91) (xy 116.84 168.91)
+		)
+		(stroke
+			(width 0)
+			(type default)
+		)
+	)
+	(wire
+		(pts
+			(xy 116.84 182.88) (xy 255.27 182.88)
 		)
 		(stroke
@@
 			(effects
 				(font
+					(size 1.27 1.27)
+				)
+				(justify right)
+			)
+		)
+		(pin "USB_DIR" output
+			(at 116.84 182.88 0)
+			(effects
+				(font
