File: hardware/d1/adc.kicad_sch (KiCad schematic)
At the start: 1 part, among them U6 ES8327

Commit message: Pre-finalize sch
Parts:
- added C35, C37, C39, C40: 100nF 16V X7R, JLCImport:CL05B104KO5NNNC, symbol JLCImport:CL05B104KO5NNNC
- added C36, C38, C41, C42, C43, C45, C46, C47, C48: 1uF 25V X5R, JLCImport:CL05A105KA5NQNC, symbol JLCImport:CL05A105KA5NQNC
- added L5, L6: BLM15AG601SN1D, JLCImport:BLM15AG601SN1D, symbol JLCImport:BLM15AG601SN1D
- added R10, R13: 10kΩ, Resistor_SMD:R_0402_1005Metric, symbol JLCImport:0402WGF1002TCE
Connections:
- net CLKIN: now reaches U6.1 (MCLK/DMIC_SDA)
- net INT/: now reaches U6.10 (INTOUT)
- net INT/: now also R10.1
- net at U6.11 (CPVDD): now also C37.1, C38.1, L6.2
- net CPTOP: now reaches U6.12 (CPTOP)
- net CPTOP: now also C46.1
- net JACK_RING_2: now reaches U6.13 (GMS0)
- net JACK_RING_2: now also C47.2
- net GND: now reaches U6.14 (CPGND)
- net GND: now also U6.22 (AGND), U6.30 (CE), U6.33 (EP), U6.4 (DGND), U6.6 (SDIN), C35.2, C36.2, C37.2, C38.2, C39.2, C40.2, C41.2, C42.2, C43.2, C45.2
- net JACK_SLEEVE: now reaches U6.15 (GMS1)
- net JACK_SLEEVE: now also C48.1
- net CPBOT: now reaches U6.16 (CPBOT)
- net CPBOT: now also C46.2
- net at U6.17 (CPVSSP): now also C45.1
- net +3V3_D: now reaches U6.2 (DVDD)
- net +3V3_D: now also C39.1
- net at U6.20 (DACVREF): now also C42.1
- net at U6.21 (AVDD): now also C35.1, C36.1, L5.1
- net at U6.23 (ADCVREF): now also C41.1
- net at U6.24 (VMID): now also C43.1
- net MIC1N: now reaches U6.25 (MIC1N)
- net MIC1N: now also C47.1
- net MIC1P: now reaches U6.26 (MIC1P)
- net MIC1P: now also C48.2
- net +1V8_D: now reaches U6.3 (PVDD)
- net +1V8_D: now also C40.1, R10.2, R13.2
- net I2C_SDA: now reaches U6.31 (CDATA)
- net I2C_SCL: now reaches U6.32 (CCLK)
- net I2S_CK: now reaches U6.5 (SCLK)
- net I2S_WS: now reaches U6.7 (LRCK)
- net I2S_SD: now reaches U6.8 (SDOUT)
- net HEADSET: now reaches U6.9 (HEADSET)
- net HEADSET: now also R13.1
- new net +1V8_CP: L6.1
- new net +3V3_A: L5.2
- no-connect marks 0 -> 5
Other:
- note added: "I2C addr: 0x18"
- note added: "SDIN grounded!"

Commit message: Fixes
Connections:
- net +1V8_D is gone; now on net +3V3_D: C40.1, R10.2, R13.2, U6.3 (PVDD)

Commit message: Fixes
Connections:
- net JACK_RING_2 renamed HP_GND
Changed lines of the file:
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@@
+		)
+	)
+	(label "HP_GND"
+		(at 38.1 151.13 0)
+		(effects
+			(font
+				(size 1.27 1.27)
+			)
+			(justify left bottom)
 		)
 	)
@@
 		)
 	)
-	(label "JACK_RING_2"
-		(at 38.1 151.13 0)
-		(effects
-			(font
-				(size 1.27 1.27)
-			)
-			(justify left bottom)
-		)
-	)
 	(label "GMS0"
 		(at 236.22 43.18 180)
@@
 		)
 	)
+	(label "HP_GND"
+		(at 248.92 43.18 0)
+		(effects
+			(font
+				(size 1.27 1.27)
+			)
+			(justify left bottom)
+		)
+	)
 	(label "I2S_WS"
 		(at 38.1 170.18 0)
-		(effects
-			(font
-				(size 1.27 1.27)
-			)
-			(justify left bottom)
-		)
-	)
-	(label "JACK_RING_2"
-		(at 248.92 43.18 0)
 		(effects
 			(font
@@
 		)
 	)
-	(hierarchical_label "JACK_RING_2"
+	(hierarchical_label "HP_GND"
 		(shape bidirectional)
 		(at 34.29 151.13 180)

Commit message: Replace parts
Parts:
- removed C35, C37, C39, C40: 100nF 16V X7R, JLCImport:CL05B104KO5NNNC, symbol JLCImport:CL05B104KO5NNNC
- added C105, C95, C96, C99: 100nF 50V, Capacitor_SMD:C_0402_1005Metric, symbol JLCImport:CL05B104KB54PNC
Connections:
- net +3V3_D: now also C95.2, C96.2
- net GND: now also C105.1, C95.1, C96.1, C99.1
- net at C38.1, L6.2, U6.11 (CPVDD): now also C99.2
- net at C36.1, L5.1, U6.21 (AVDD): now also C105.2
