File: hardware/d1/power.kicad_sch (KiCad schematic)
At the start: 44 parts, among them U10 BLM15PX601SN1D, U11 TPS7A2033PDBVR, U12 TPS7A2018PDBVR, U13 TPS7A2018PDBVR, U7 TPS7A2018PDBVR, U8 TPS7A2033PDBVR, U9 TPS560430XFDBVR

Commit message: Replace parts
Parts:
- removed C1: 100nF 16V X7R, JLCImport:CL05B104KO5NNNC, symbol JLCImport:CL05B104KO5NNNC
- removed C13: 4.7uF 10V X5R, JLCImport:CL05A475MP5NRNC, symbol JLCImport:CL05A475MP5NRNC
- removed C3: 4.7uF 10V X5R, Capacitor_SMD:C_0603_1608Metric, symbol JLCImport:CL10A475KP8NNNC
- removed C86: 100nF 50V X7R, Capacitor_SMD:C_0402_1005Metric, symbol JLCImport:CC0402KRX7R9BB104
- added C35, C40: 4.7uF 16V, Capacitor_SMD:C_0603_1608Metric, symbol JLCImport:CL10A475KO8NNNC
- added C79, C86: 100nF 50V, Capacitor_SMD:C_0402_1005Metric, symbol JLCImport:CL05B104KB54PNC
Connections:
- net +1V8_CP: now also C40.2
- net +1V8_D: now also C35.2
- net GND: now also C35.1, C40.1, C86.1
- net PWR_IN: now also C86.2
- net at L2.1, U9.6 (SW): now also C79.2
- net at U9.1 (CB): now also C79.1
