File: hardware/d1/power.kicad_sch (KiCad schematic)
At the start: 44 parts, among them U10 BLM15PX601SN1D, U11 TPS7A2033PDBVR, U12 TPS7A2018PDBVR, U13 TPS7A2018PDBVR, U7 TPS7A2018PDBVR, U8 TPS7A2033PDBVR, U9 TPS560430XFDBVR

Commit message: Traces
Connections:
- net GND: now also U11.4 (NC), U12.4 (N/C), U13.4 (N/C), U7.4 (N/C), U8.4 (NC)
- no-connect marks 5 -> 0
Changed lines of the file:
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@@
+	)
+	(junction
+		(at 134.62 111.76)
+		(diameter 0)
+		(color 0 0 0 0)
 	)
 	(junction
@@
 	)
 	(junction
+		(at 133.35 165.1)
+		(diameter 0)
+		(color 0 0 0 0)
+	)
+	(junction
 		(at 81.28 50.8)
 		(diameter 0)
@@
 	)
 	(junction
+		(at 64.77 166.37)
+		(diameter 0)
+		(color 0 0 0 0)
+	)
+	(junction
 		(at 152.4 44.45)
 		(diameter 0)
@@
 	)
 	(junction
+		(at 66.04 113.03)
+		(diameter 0)
+		(color 0 0 0 0)
+	)
+	(junction
 		(at 45.72 113.03)
 		(diameter 0)
@@
 	)
 	(junction
+		(at 187.96 111.76)
+		(diameter 0)
+		(color 0 0 0 0)
+	)
+	(junction
 		(at 59.69 50.8)
 		(diameter 0)
@@
 		(color 0 0 0 0)
 	)
-	(no_connect
-		(at 133.35 160.02)
-	)
-	(no_connect
-		(at 134.62 106.68)
-	)
-	(no_connect
-		(at 187.96 105.41)
-	)
-	(no_connect
-		(at 66.04 105.41)
-	)
-	(no_connect
-		(at 64.77 158.75)
-	)
 	(wire
 		(pts
@@
 	(wire
 		(pts
+			(xy 187.96 105.41) (xy 187.96 111.76)
+		)
+		(stroke
+			(width 0)
+			(type default)
+		)
+	)
+	(wire
+		(pts
 			(xy 114.3 25.4) (xy 115.57 25.4)
 		)
@@
 	(wire
 		(pts
+			(xy 133.35 160.02) (xy 133.35 165.1)
+		)
+		(stroke
+			(width 0)
+			(type default)
+		)
+	)
+	(wire
+		(pts
 			(xy 44.45 146.05) (xy 44.45 152.4)
 		)
@@
 	(wire
 		(pts
+			(xy 66.04 113.03) (xy 69.85 113.03)
+		)
+		(stroke
+			(width 0)
+			(type default)
+		)
+	)
+	(wire
+		(pts
 			(xy 167.64 44.45) (xy 172.72 44.45)
 		)
@@
 	(wire
 		(pts
+			(xy 133.35 165.1) (xy 137.16 165.1)
+		)
+		(stroke
+			(width 0)
+			(type default)
+		)
+	)
+	(wire
+		(pts
 			(xy 107.95 160.02) (xy 107.95 154.94)
 		)
@@
 	(wire
 		(pts
-			(xy 45.72 113.03) (xy 69.85 113.03)
+			(xy 45.72 113.03) (xy 66.04 113.03)
 		)
 		(stroke
@@
 	(wire
 		(pts
-			(xy 111.76 165.1) (xy 137.16 165.1)
+			(xy 111.76 165.1) (xy 133.35 165.1)
 		)
 		(stroke
@@
 	(wire
 		(pts
-			(xy 55.88 166.37) (xy 68.58 166.37)
+			(xy 55.88 166.37) (xy 64.77 166.37)
 		)
 		(stroke
@@
 	(wire
 		(pts
+			(xy 64.77 166.37) (xy 68.58 166.37)
+		)
+		(stroke
+			(width 0)
+			(type default)
+		)
+	)
+	(wire
+		(pts
 			(xy 191.77 110.49) (xy 191.77 111.76)
 		)
@@
 	(wire
 		(pts
-			(xy 138.43 111.76) (xy 125.73 111.76)
+			(xy 138.43 111.76) (xy 134.62 111.76)
 		)
 		(stroke
@@
 	(wire
 		(pts
+			(xy 134.62 106.68) (xy 134.62 111.76)
+		)
+		(stroke
+			(width 0)
+			(type default)
+		)
+	)
+	(wire
+		(pts
 			(xy 53.34 38.1) (xy 57.15 38.1)
 		)
@@
 	(wire
 		(pts
+			(xy 134.62 111.76) (xy 125.73 111.76)
+		)
+		(stroke
+			(width 0)
+			(type default)
+		)
+	)
+	(wire
+		(pts
 			(xy 138.43 93.98) (xy 144.78 93.98)
 		)
@@
 	(wire
 		(pts
+			(xy 187.96 111.76) (xy 179.07 111.76)
+		)
+		(stroke
+			(width 0)
+			(type default)
+		)
+	)
+	(wire
+		(pts
 			(xy 113.03 160.02) (xy 107.95 160.02)
 		)
@@
 	(wire
 		(pts
+			(xy 66.04 105.41) (xy 66.04 113.03)
+		)
+		(stroke
+			(width 0)
+			(type default)
+		)
+	)
+	(wire
+		(pts
 			(xy 40.64 152.4) (xy 44.45 152.4)
 		)
@@
 	(wire
 		(pts
-			(xy 191.77 111.76) (xy 179.07 111.76)
+			(xy 191.77 111.76) (xy 187.96 111.76)
 		)
 		(stroke
@@
 		)
 		(stroke
+			(width 0)
+			(type default)
+		)
+	)
+	(wire
+		(pts
+			(xy 64.77 158.75) (xy 64.77 166.37)
+		)
+		(stroke

Commit message: Almost done tracing
Parts:
- removed C63: 47uF 25V X5R, Capacitor_SMD:C_1206_3216Metric, symbol JLCImport:C3216X5R1E476MTJ00E
Changed lines of the file:
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@@
 	)
 	(junction
-		(at 167.64 36.83)
-		(diameter 0)
-		(color 0 0 0 0)
-	)
-	(junction
 		(at 166.37 107.95)
 		(diameter 0)
@@
 	)
 	(junction
-		(at 167.64 44.45)
-		(diameter 0)
-		(color 0 0 0 0)
-	)
-	(junction
 		(at 191.77 92.71)
 		(diameter 0)
@@
 	(wire
 		(pts
-			(xy 167.64 44.45) (xy 172.72 44.45)
-		)
-		(stroke
-			(width 0)
-			(type default)
-		)
-	)
-	(wire
-		(pts
 			(xy 81.28 50.8) (xy 87.63 50.8)
 		)
@@
 	(wire
 		(pts
-			(xy 167.64 36.83) (xy 172.72 36.83)
-		)
-		(stroke
-			(width 0)
-			(type default)
-		)
-	)
-	(wire
-		(pts
 			(xy 134.62 106.68) (xy 134.62 111.76)
 		)
@@
 		(property "Value" "47uF 25V X5R"
 			(at 169.164 42.164 0)
+			(hide yes)
 			(show_name no)
 			(do_not_autoplace no)
@@
 					(unit 1)
 				)
-			)
-		)
-	)
-	(symbol
-		(lib_id "JLCImport:C3216X5R1E476MTJ00E")
-		(at 172.72 40.64 90)
-		(unit 1)
-		(body_style 1)
-		(exclude_from_sim no)
-		(in_bom yes)
-		(on_board yes)
-		(in_pos_files yes)
-		(dnp yes)
-		(property "Reference" "C63"
-			(at 171.45 41.91 0)
-			(show_name no)
-			(do_not_autoplace no)
-			(effects
-				(font
-					(size 1.27 1.27)
-				)
-				(justify right)
-			)
-		)
-		(property "Value" "47uF 25V X5R"
-			(at 174.244 42.164 0)
-			(show_name no)
-			(do_not_autoplace no)
-			(effects
-				(font
-					(size 1.27 1.27)
-				)
-				(justify right)
-			)
-		)
-		(property "Footprint" "Capacitor_SMD:C_1206_3216Metric"
-			(at 172.72 40.64 0)
-			(hide yes)
-			(show_name no)
-			(do_not_autoplace no)
-			(effects
-				(font
-					(size 1.27 1.27)
-				)
-			)
-		)
-		(property "Datasheet" "https://www.lcsc.com/datasheet/lcsc_datasheet_2304140030_TDK-C3216X5R1E476MTJ00E_C76659.pdf"
-			(at 172.72 40.64 0)
-			(hide yes)
-			(show_name no)
-			(do_not_autoplace no)
-			(effects
-				(font
-					(size 1.27 1.27)
-				)
-			)
-		)
-		(property "Description" "25V 47uF X5R ±20% 1206 Multilayer Ceramic Capacitors MLCC - SMD/SMT ROHS"
-			(at 172.72 40.64 0)
-			(hide yes)
-			(show_name no)
-			(do_not_autoplace no)
-			(effects
-				(font
-					(size 1.27 1.27)
-				)
-			)
-		)
-		(property "LCSC" "C76659"
-			(at 172.72 40.64 0)
-			(hide yes)
-			(show_name no)
-			(do_not_autoplace no)
-			(effects
-				(font
-					(size 1.27 1.27)
-				)
-			)
-		)
-		(property "Manufacturer" "TDK"
-			(at 172.72 40.64 0)
-			(hide yes)
-			(show_name no)
-			(do_not_autoplace no)
-			(effects
-				(font
-					(size 1.27 1.27)
-				)
-			)
-		)
-		(property "Manufacturer Part" "C3216X5R1E476MTJ00E"
-			(at 172.72 40.64 0)
-			(hide yes)
-			(show_name no)
-			(do_not_autoplace no)
-			(effects
-				(font
-					(size 1.27 1.27)
-				)
-			)
-		)
-		(pin "1"
-		)
-		(pin "2"
-		)
-		(instances
-			(project "DrunkEarPhoneAdapter"
-				(path "/df940915-8af0-46f9-b18a-23d4684ae671/bea21a31-aee1-46f9-b13e-ece764487360"
-					(reference "C63")
-					(unit 1)
-				)

Commit message: Fix track lengths
Parts:
- added TP8: GND, TestPoint:TestPoint_Pad_1.0x1.0mm, symbol Connector:TestPoint
Connections:
- net GND: now also TP8.1
Changed lines of the file:
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@@
 	)
 	(junction
+		(at 93.98 63.5)
+		(diameter 0)
+		(color 0 0 0 0)
+	)
+	(junction
 		(at 133.35 165.1)
 		(diameter 0)
@@
 	(wire
 		(pts
+			(xy 93.98 63.5) (xy 100.33 63.5)
+		)
+		(stroke
+			(width 0)
+			(type default)
+		)
+	)
+	(wire
+		(pts
 			(xy 57.15 48.26) (xy 60.96 48.26)
 		)
@@
 					(unit 1)
 				)
+			)
+		)
+	)
+	(symbol
+		(lib_id "Connector:TestPoint")
+		(at 100.33 63.5 0)
+		(unit 1)
+		(body_style 1)
+		(exclude_from_sim no)
+		(in_bom yes)
+		(on_board yes)
+		(in_pos_files yes)
+		(dnp no)
+		(fields_autoplaced yes)
+		(property "Reference" "TP8"
+			(at 102.87 58.9279 0)
+			(show_name no)
+			(do_not_autoplace no)
+			(effects
+				(font
+					(size 1.27 1.27)
+				)
+				(justify left)
+			)
+		)
+		(property "Value" "GND"
+			(at 102.87 61.4679 0)
+			(show_name no)
+			(do_not_autoplace no)
+			(effects
+				(font
+					(size 1.27 1.27)
+				)
+				(justify left)
+			)
+		)
+		(property "Footprint" "TestPoint:TestPoint_Pad_1.0x1.0mm"
+			(at 105.41 63.5 0)
+			(hide yes)
+			(show_name no)
+			(do_not_autoplace no)
+			(effects
+				(font
+					(size 1.27 1.27)
+				)
+			)
+		)
+		(property "Datasheet" ""
+			(at 105.41 63.5 0)
+			(hide yes)
+			(show_name no)
+			(do_not_autoplace no)
+			(effects
+				(font
+					(size 1.27 1.27)
+				)
+			)
+		)
+		(property "Description" "test point"
+			(at 100.33 63.5 0)
+			(hide yes)
+			(show_name no)
+			(do_not_autoplace no)
+			(effects
+				(font
+					(size 1.27 1.27)
+				)
+			)
+		)
+		(pin "1"
+		)
+		(instances
+			(project "DrunkEarPhoneAdapter"
+				(path "/df940915-8af0-46f9-b18a-23d4684ae671/bea21a31-aee1-46f9-b13e-ece764487360"
+					(reference "TP8")
+					(unit 1)
+				)

Commit message: Route fixes
Changed lines of the file:
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@@
 	)
 	(junction
-		(at 87.63 50.8)
+		(at 157.48 44.45)
 		(diameter 0)
 		(color 0 0 0 0)
 	)
 	(junction
-		(at 157.48 44.45)
+		(at 87.63 50.8)
 		(diameter 0)
 		(color 0 0 0 0)
@@
 	)
 	(junction
-		(at 87.63 49.53)
-		(diameter 0)
-		(color 0 0 0 0)
-	)
-	(junction
 		(at 57.15 113.03)
 		(diameter 0)
@@
 	(wire
 		(pts
-			(xy 81.28 62.23) (xy 81.28 63.5)
-		)
-		(stroke
-			(width 0)
-			(type default)
-		)
-	)
-	(wire
-		(pts
-			(xy 87.63 48.26) (xy 87.63 49.53)
-		)
-		(stroke
-			(width 0)
-			(type default)
-		)
-	)
-	(wire
-		(pts
 			(xy 133.35 160.02) (xy 133.35 165.1)
 		)
@@
 	(wire
 		(pts
+			(xy 87.63 50.8) (xy 87.63 54.61)
+		)
+		(stroke
+			(width 0)
+			(type default)
+		)
+	)
+	(wire
+		(pts
 			(xy 24.13 57.15) (xy 34.29 57.15)
 		)
@@
 	(wire
 		(pts
-			(xy 87.63 49.53) (xy 87.63 54.61)
-		)
-		(stroke
-			(width 0)
-			(type default)
-		)
-	)
-	(wire
-		(pts
 			(xy 93.98 62.23) (xy 93.98 63.5)
 		)
@@
 	(wire
 		(pts
+			(xy 87.63 50.8) (xy 96.52 50.8)
+		)
+		(stroke
+			(width 0)
+			(type default)
+		)
+	)
+	(wire
+		(pts
 			(xy 109.22 99.06) (xy 113.03 99.06)
 		)
@@
 	(wire
 		(pts
+			(xy 87.63 48.26) (xy 87.63 50.8)
+		)
+		(stroke
+			(width 0)
+			(type default)
+		)
+	)
+	(wire
+		(pts
 			(xy 142.24 36.83) (xy 147.32 36.83)
 		)
@@
 	(wire
 		(pts
-			(xy 87.63 50.8) (xy 96.52 50.8)
-		)
-		(stroke
-			(width 0)
-			(type default)
-		)
-	)
-	(wire
-		(pts
 			(xy 157.48 36.83) (xy 162.56 36.83)
 		)
@@
 	(symbol
 		(lib_id "power:+5V")
-		(at 87.63 49.53 0)
+		(at 87.63 48.26 0)
 		(unit 1)
 		(body_style 1)
@@
 		(fields_autoplaced yes)
 		(property "Reference" "#PWR022"
-			(at 87.63 53.34 0)
+			(at 87.63 52.07 0)
 			(hide yes)
 			(show_name no)
@@
 		)
 		(property "Value" "PWR_IN"
-			(at 87.63 44.45 0)
+			(at 87.63 43.18 0)
 			(show_name no)
 			(do_not_autoplace no)
@@
 		)
 		(property "Footprint" ""
-			(at 87.63 49.53 0)
+			(at 87.63 48.26 0)
 			(hide yes)
 			(show_name no)
@@
 		)
 		(property "Datasheet" ""
-			(at 87.63 49.53 0)
+			(at 87.63 48.26 0)
 			(hide yes)
 			(show_name no)
@@
 		)
 		(property "Description" "Power symbol creates a global label with name \"+5V\""
-			(at 87.63 49.53 0)
+			(at 87.63 48.26 0)
 			(hide yes)
 			(show_name no)
