File: hardware/d1/ucpd.kicad_sch (KiCad schematic)
At the start: 3 parts, among them U4 TCPP03-M20, U5 TCPP03-M20

Commit message: Pre-finalize sch
Parts:
- added C44, C74: 100nF 16V X7R, JLCImport:CL05B104KO5NNNC, symbol JLCImport:CL05B104KO5NNNC
- added C66: 10nF 50V X7R, Capacitor_SMD:C_0402_1005Metric, symbol JLCImport:CL05B103KB5NNNC
- added C67, C68: 2.2uF 50V X7R, JLCImport:CC0805KKX7R9BB225, symbol JLCImport:CC0805KKX7R9BB225
- added C69, C75: 100nF 50V X7R, JLCImport:CL05B104KB54PNC, symbol JLCImport:CL05B104KB54PNC
- added C70, C71, C72, C73: 330pF 50V, Capacitor_SMD:C_0402_1005Metric, symbol JLCImport:CL05C331JB5NNNC
- added D1, D3: PMEG4010CEH_115, Diode_SMD:D_SOD-110, symbol JLCImport:PMEG4010CEH_115
- added L7: ECMF02-2AMX6, JLCImport:ECMF02-2AMX6, symbol JLCImport:ECMF02-2AMX6
- added Q1, Q2: CSD17577Q3A, JLCImport:CSD17577Q3A, symbol JLCImport:CSD17577Q3A
- added R17, R18: 10mΩ 500mW, Resistor_SMD:R_0805_2012Metric, symbol JLCImport:ERJ6BWFR010V
- added R19, R22, R26, R29: 10kΩ, Resistor_SMD:R_0402_1005Metric, symbol JLCImport:0402WGF1002TCE
- added R20, R27: 560Ω, Resistor_SMD:R_0402_1005Metric, symbol JLCImport:0402WGF5600TCE
- added R21, R28: 130kΩ, Resistor_SMD:R_0402_1005Metric, symbol JLCImport:RC0402FR-07130KL
- added R23, R30: 0Ω, Resistor_SMD:R_0402_1005Metric, symbol JLCImport:RC0402FR-070RL
- added R24, R25: 47kΩ, Resistor_SMD:R_0402_1005Metric, symbol JLCImport:0402WGF4702TCE
- added U15, U16: ESDA25P35-1U1M, JLCImport:ESDA25P35-1U1M_C19829649, symbol JLCImport:ESDA25P35-1U1M_C19829649
- added USBC2: (no value), JLCImport:USBC_EXT_5P, symbol JLCImport:USBC_5P_EXT
Connections:
- net USB_CHR_CC1: now also U5.15 (CC1c), C70.2
- net USB_CHR_CC2: now also U5.13 (CC2c), C71.2
- net USB_CHR_VBUS: now also U5.9 (VBUSc), C67.1, R17.1, R26.2, R28.2, U16.1 (C)
- net UCPD2_CC1: now reaches U5.1 (CC1)
- net USB_CHR_ISENSE: now reaches U5.10 (Isense)
- net USB_CHR_ISENSE: now also D1.2 (A), Q1.5 (D), Q1.6 (D), Q1.7 (D), Q1.8 (D), Q1.9 (D), R17.2
- net VSENSE_CHR: now reaches U5.11 (Vsense)
- net VSENSE_CHR: now also R26.1, R27.2
- net +3V3_D: now reaches U5.12 (GND)
- net +3V3_D: now also U4.12 (GND), U4.16 (I2C_ADD), U4.2 (VCC_VCONN), U4.21 (GND), U5.2 (VCC_VCONN), U5.21 (GND), USBC1.0, USBC1.A1 (GND), USBC1.A12 (GND), USBC1.B1 (GND), USBC1.B12 (GND), C44.1, C44.2, C67.2, C68.2, C69.2, C70.1, C71.1, C72.1, C73.1, C74.1, C74.2, C75.2, L7.3 (GND), R20.1, R22.1, R27.1, R29.1, U15.2 (A), U16.2 (A), USBC2.5 (GND)
- net at U5.14 (CBIAS): now also C75.1
- net +1V8_D: now reaches U5.16 (I2C_ADD)
- net +1V8_D: now also U4.20 (EN), U5.20 (EN), R24.2, R25.2
- net I2C1_SDA: now reaches U5.17 (SDA)
- net I2C1_SDA: now also U4.17 (SDA)
- net I2C1_SCL: now reaches U5.18 (SCL)
- net I2C1_SCL: now also U4.18 (SCL)
- net CHR_INT/: now reaches U5.19 (FLGn)
- net CHR_INT/: now also R25.1
- net UCPD2_CC2: now reaches U5.3 (CC2)
- net at U5.4 (IANA): now also R30.2
- net UCPD1_CC1: now reaches U4.1 (CC1)
- net USB_PHONE_ISENSE: now reaches U4.10 (Isense)
- net USB_PHONE_ISENSE: now also D3.2 (A), Q2.5 (D), Q2.6 (D), Q2.7 (D), Q2.8 (D), Q2.9 (D), R18.2
- net VSENSE_PHONE: now reaches U4.11 (Vsense)
- net VSENSE_PHONE: now also R19.1, R20.2
- net USB_PHONE_CC2: now reaches U4.13 (CC2c)
- net USB_PHONE_CC2: now also C73.2
- net at U4.14 (CBIAS): now also C69.1
- net USB_PHONE_CC1: now reaches U4.15 (CC1c)
- net USB_PHONE_CC1: now also C72.2, USBC2.4 (CC)
- net PHONE_INT/: now reaches U4.19 (FLGn)
- net PHONE_INT/: now also R24.1
- net UCPD1_CC2: now reaches U4.3 (CC2)
- net at U4.4 (IANA): now also R23.2
- net GDPg: now reaches U4.5 (GDPg)
- net GDPg: now also C66.2, Q1.4 (G), Q2.4 (G)
- net GDPs: now reaches U4.6 (GDPs)
- net GDPs: now also C66.1, Q1.1 (S), Q1.2 (S), Q1.3 (S), Q2.1 (S), Q2.2 (S), Q2.3 (S)
- net USB_PHONE_VBUS: now reaches U4.9 (VBUSc)
- net USB_PHONE_VBUS: now also C68.1, R18.1, R19.2, R21.2, U15.1 (C), USBC2.1 (VBUS)
- new net: L7.5 (D-), USBC2.2 (D-)
- new net: L7.6 (D+), USBC2.3 (D+)
- new net ADC_CHR_IANA: R30.1
- new net ADC_CHR_VBUS: R28.1, R29.2
- new net ADC_PHONE_IANA: R23.1
- new net ADC_PHONE_VBUS: R21.1, R22.2
- new net PWR_IN: D1.1 (K), D3.1 (K)
- new net USB_DN: L7.2 (D-)
- new net USB_DP: L7.1 (D+)
- no-connect marks 10 -> 17
Other:
- note added: "Charger side"
- note added: "I2C addr: 0x34"
- note added: "I2C addr: 0x35"
- note added: "Phone side"
- moved on the sheet: U4, U5, USBC1

Commit message: Fix issue, add exti
Connections:
- net +3V3_D: no longer C44.2, C67.2, C68.2, C69.2, C70.1, C71.1, C72.1, C73.1, C74.2, C75.2, L7.3 (GND), R20.1, R22.1, R27.1, R29.1, U15.2 (A), U16.2 (A), U4.12 (GND), U4.16 (I2C_ADD), U4.21 (GND), U5.12 (GND), U5.21 (GND), USBC1.0, USBC1.A1 (GND), USBC1.A12 (GND), USBC1.B1 (GND), USBC1.B12 (GND), USBC2.5 (GND)
- new net GND: C44.2, C67.2, C68.2, C69.2, C70.1, C71.1, C72.1, C73.1, C74.2, C75.2, L7.3 (GND), R20.1, R22.1, R27.1, R29.1, U15.2 (A), U16.2 (A), U4.12 (GND), U4.16 (I2C_ADD), U4.21 (GND), U5.12 (GND), U5.21 (GND), USBC1.0, USBC1.A1 (GND), USBC1.A12 (GND), USBC1.B1 (GND), USBC1.B12 (GND), USBC2.5 (GND)
Changed lines of the file:
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@@
-	)
-	(junction
-		(at 168.91 96.52)
-		(diameter 0)
-		(color 0 0 0 0)
 	)
 	(junction
@@
 		)
 		(stroke
-			(width 0)
-			(type default)
-		)
-	)
-	(wire
-		(pts
-			(xy 168.91 86.36) (xy 168.91 96.52)
-		)
-		(stroke

Commit message: Fixes
Parts:
- removed C69, C75: 100nF 50V X7R, JLCImport:CL05B104KB54PNC, symbol JLCImport:CL05B104KB54PNC
- added C80, C81, C82, C83: 1nF 50V X7R, Capacitor_SMD:C_0402_1005Metric, symbol JLCImport:CL05B102KB5NNNC
- added C87, C88: 100nF 50V X7R, Capacitor_SMD:C_0402_1005Metric, symbol JLCImport:CC0402KRX7R9BB104
- D1, D3: footprint Diode_SMD:D_SOD-110 -> Diode_SMD:D_SOD-123F
Connections:
- net ADC_CHR_IANA: now also C83.2
- net ADC_CHR_VBUS: now also C80.2
- net ADC_PHONE_IANA: now also C82.2
- net ADC_PHONE_VBUS: now also C81.2
- net GND: now also C80.1, C81.1, C82.1, C83.1, C87.1, C88.1
- net at U4.14 (CBIAS): now also C87.2
- net at U5.14 (CBIAS): now also C88.2
Other:
- moved on the sheet: R26, R27, R28, R29

Commit message: Fixes
Parts:
- added R36: 100kΩ, JLCImport:0402WGF1003TCE, symbol JLCImport:0402WGF1003TCE
Connections:
- net +3V3_D: now also R24.2, R25.2, U5.16 (I2C_ADD), U5.20 (EN)
- net GND: now also R36.1
- removed net +1V8_D: R24.2, R25.2, U4.20 (EN), U5.16 (I2C_ADD), U5.20 (EN)
- new net PHONE_EN: R36.2, U4.20 (EN)
Other:
- note added: "Disabled by default"

Commit message: Fixesss
Parts:
- USBC2: now left out of the parts list
Changed lines of the file:
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@@
 		(body_style 1)
 		(exclude_from_sim no)
-		(in_bom yes)
+		(in_bom no)
 		(on_board yes)
-		(in_pos_files yes)
+		(in_pos_files no)
 		(dnp no)
 		(fields_autoplaced yes)

Commit message: Fixes
Parts:
- removed C67, C68: 2.2uF 50V X7R, JLCImport:CC0805KKX7R9BB225, symbol JLCImport:CC0805KKX7R9BB225
- removed R19, R26: 10kΩ, Resistor_SMD:R_0402_1005Metric, symbol JLCImport:0402WGF1002TCE
- removed R20, R27: 560Ω, Resistor_SMD:R_0402_1005Metric, symbol JLCImport:0402WGF5600TCE
- added C64, C65: 2.2uF 50V X7R, Capacitor_SMD:C_1206_3216Metric, symbol JLCImport:CL31B225KBHNNNE
- added C84: 100nF 16V X7R, JLCImport:CL05B104KO5NNNC, symbol JLCImport:CL05B104KO5NNNC
- added JP2, JP3, JP4: SolderJumper_2_Bridged, Jumper:SolderJumper-2_P1.3mm_Bridged_RoundedPad1.0x1.5mm, symbol Jumper:SolderJumper_2_Bridged
- added L8: ECMF02-2AMX6, JLCImport:ECMF02-2AMX6, symbol JLCImport:ECMF02-2AMX6
- added R19, R20: 510Ω, Resistor_SMD:R_0603_1608Metric, symbol JLCImport:0603WAJ0511T5E
- added R40, R41: 10kΩ 0603, Resistor_SMD:R_0603_1608Metric, symbol JLCImport:RC0603FR-0710KL
- added R42: 100kΩ, JLCImport:0402WGF1003TCE, symbol JLCImport:0402WGF1003TCE
- added U3: TS3USB221RSER, JLCImport:TS3USB221RSER, symbol JLCImport:TS3USB221RSER
Connections:
- net +3V3_D: now also C84.1, U3.10 (VCC)
- net GDPs: no longer C66.1
- net GND: now also C64.1, C65.1, C84.2, L8.3 (GND), R19.1, R20.1, R42.1, U3.5 (GND), U3.6 (OE#)
- net USB_CHR_DN: now also L8.2 (D-)
- net USB_CHR_DP: now also L8.1 (D+)
- net USB_CHR_ISENSE: now also JP3.2 (B), JP4.2 (B)
- net USB_CHR_VBUS: now also C65.2, R41.2
- net USB_DN: now also U3.2 (1D-); no longer L7.2 (D-)
- net USB_DP: now also U3.1 (1D+); no longer L7.1 (D+)
- net USB_PHONE_ISENSE: now also C66.1, JP2.2 (B)
- net USB_PHONE_VBUS: now also C64.2, R40.2
- net VSENSE_CHR: now also R20.2, R41.1
- net VSENSE_PHONE: now also R19.2, R40.1
- net GDPs_CHR: now reaches U5.6 (GDPs)
- net GDPs_CHR: now also JP4.1 (A)
- net GDCs_CHR: now reaches U5.8 (GDCs)
- net GDCs_CHR: now also JP3.1 (A)
- net GDCs: now reaches U4.8 (GDCs)
- net GDCs: now also JP2.1 (A)
- new net USB_CHR_SAFE_DN: L8.5 (D-), U3.4 (2D-)
- new net USB_CHR_SAFE_DP: L8.6 (D+), U3.3 (2D+)
- new net USB_DIR: R42.2, U3.9 (S)
- new net USB_PHONE_SAFE_DN: L7.2 (D-), U3.7 (D-)
- new net USB_PHONE_SAFE_DP: L7.1 (D+), U3.8 (D+)
- no-connect marks 17 -> 15
Other:
- note added: "ESD"
- note added: "USB bypass switch"
- note added: "Unused mosfet channels"
- moved on the sheet: L7, USBC2

Commit message: Fixes
Parts:
- removed R19, R20: 510Ω, Resistor_SMD:R_0603_1608Metric, symbol JLCImport:0603WAJ0511T5E
- added R19, R20: 549Ω, Resistor_SMD:R_0603_1608Metric, symbol JLCImport:0603WAF5490T5E
Connections:
- net GND: now also R19.1, R20.1
- net VSENSE_CHR: now also R20.2
- net VSENSE_PHONE: now also R19.2
Changed lines of the file:
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@@
 	)
 	(junction
+		(at 137.16 133.35)
+		(diameter 0)
+		(color 0 0 0 0)
+	)
+	(junction
 		(at 35.56 48.26)
 		(diameter 0)
@@
 	)
 	(junction
-		(at 137.16 133.35)
-		(diameter 0)
-		(color 0 0 0 0)
-	)
-	(junction
 		(at 27.94 124.46)
 		(diameter 0)
@@
 	)
 	(junction
-		(at 16.51 134.62)
+		(at 17.78 87.63)
 		(diameter 0)
 		(color 0 0 0 0)
 	)
 	(junction
-		(at 17.78 87.63)
+		(at 36.83 144.78)
 		(diameter 0)
 		(color 0 0 0 0)
 	)
 	(junction
-		(at 36.83 144.78)
+		(at 101.6 36.83)
 		(diameter 0)
 		(color 0 0 0 0)
 	)
 	(junction
-		(at 101.6 36.83)
+		(at 16.51 134.62)
 		(diameter 0)
 		(color 0 0 0 0)
@@
 	)
 	(symbol
-		(lib_id "JLCImport:0603WAJ0511T5E")
-		(at 16.51 139.7 90)
+		(lib_id "JLCImport:0603WAF5490T5E")
+		(at 137.16 138.43 90)
 		(unit 1)
 		(body_style 1)
@@
 		(dnp no)
 		(fields_autoplaced yes)
-		(property "Reference" "R19"
-			(at 19.05 138.4299 90)
+		(property "Reference" "R20"
+			(at 139.7 137.1599 90)
 			(show_name no)
 			(do_not_autoplace no)
@@
 			)
 		)
-		(property "Value" "510Ω"
-			(at 19.05 140.9699 90)
+		(property "Value" "549Ω"
+			(at 139.7 139.6999 90)
 			(show_name no)
 			(do_not_autoplace no)
@@
 		)
 		(property "Footprint" "Resistor_SMD:R_0603_1608Metric"
-			(at 16.51 139.7 0)
+			(at 137.16 138.43 0)
 			(hide yes)
 			(show_name no)
@@
 			)
 		)
-		(property "Datasheet" "https://www.lcsc.com/datasheet/lcsc_datasheet_2205311845_UNI-ROYAL-Uniroyal-Elec-0603WAJ0511T5E_C25245.pdf"
-			(at 16.51 139.7 0)
+		(property "Datasheet" "https://www.lcsc.com/datasheet/lcsc_datasheet_2206010116_UNI-ROYAL-Uniroyal-Elec-0603WAF5490T5E_C23079.pdf"
+			(at 137.16 138.43 0)
 			(hide yes)
 			(show_name no)
@@
 			)
 		)
-		(property "Description" "-55℃~+155℃ 100mW 510Ω 75V Thick Film Resistor ±100ppm/℃ ±5% 0603 Chip Resistor - Surface Mount ROHS"
-			(at 16.51 139.7 0)
+		(property "Description" "-55℃~+155℃ 100mW 549Ω 75V Thick Film Resistor ±1% ±100ppm/℃ 0603 Chip Resistor - Surface Mount ROHS"
+			(at 137.16 138.43 0)
 			(hide yes)
 			(show_name no)
@@
 			)
 		)
-		(property "LCSC" "C25245"
-			(at 16.51 139.7 0)
+		(property "LCSC" "C23079"
+			(at 137.16 138.43 0)
 			(hide yes)
 			(show_name no)
@@
 		)
 		(property "Manufacturer" "UNI-ROYAL(Uniroyal Elec)"
-			(at 16.51 139.7 0)
+			(at 137.16 138.43 0)
 			(hide yes)
 			(show_name no)
@@
 			)
 		)
-		(property "Manufacturer Part" "0603WAJ0511T5E"
-			(at 16.51 139.7 0)
+		(property "Manufacturer Part" "0603WAF5490T5E"
+			(at 137.16 138.43 0)
 			(hide yes)
 			(show_name no)
@@
 			(project "DrunkEarPhoneAdapter"
 				(path "/df940915-8af0-46f9-b18a-23d4684ae671/5c561383-fdd0-44ae-83ac-568aac0f03a9"
-					(reference "R19")
+					(reference "R20")
 					(unit 1)
 				)
@@
 	)
 	(symbol
+		(lib_id "JLCImport:0603WAF5490T5E")
+		(at 16.51 139.7 90)
+		(unit 1)
+		(body_style 1)
+		(exclude_from_sim no)
+		(in_bom yes)
+		(on_board yes)
+		(in_pos_files yes)
+		(dnp no)
+		(fields_autoplaced yes)
+		(property "Reference" "R19"
+			(at 19.05 138.4299 90)
+			(show_name no)
+			(do_not_autoplace no)
+			(effects
+				(font
+					(size 1.27 1.27)
+				)
+				(justify right)
+			)
+		)
+		(property "Value" "549Ω"
+			(at 19.05 140.9699 90)
+			(show_name no)
+			(do_not_autoplace no)
+			(effects
+				(font
+					(size 1.27 1.27)
+				)
+				(justify right)
+			)
+		)
+		(property "Footprint" "Resistor_SMD:R_0603_1608Metric"
+			(at 16.51 139.7 0)
+			(hide yes)
+			(show_name no)
+			(do_not_autoplace no)
+			(effects
+				(font
+					(size 1.27 1.27)
+				)
+			)
+		)
+		(property "Datasheet" "https://www.lcsc.com/datasheet/lcsc_datasheet_2206010116_UNI-ROYAL-Uniroyal-Elec-0603WAF5490T5E_C23079.pdf"
+			(at 16.51 139.7 0)
+			(hide yes)
+			(show_name no)
+			(do_not_autoplace no)
+			(effects
+				(font
+					(size 1.27 1.27)
+				)
+			)
+		)
+		(property "Description" "-55℃~+155℃ 100mW 549Ω 75V Thick Film Resistor ±1% ±100ppm/℃ 0603 Chip Resistor - Surface Mount ROHS"
+			(at 16.51 139.7 0)
+			(hide yes)
+			(show_name no)
+			(do_not_autoplace no)
+			(effects
+				(font
+					(size 1.27 1.27)
+				)
+			)
+		)
+		(property "LCSC" "C23079"
+			(at 16.51 139.7 0)
+			(hide yes)
+			(show_name no)
+			(do_not_autoplace no)
+			(effects
+				(font
+					(size 1.27 1.27)
+				)
+			)
+		)
+		(property "Manufacturer" "UNI-ROYAL(Uniroyal Elec)"
+			(at 16.51 139.7 0)
+			(hide yes)
+			(show_name no)
+			(do_not_autoplace no)
+			(effects
+				(font
+					(size 1.27 1.27)
+				)
+			)
+		)
+		(property "Manufacturer Part" "0603WAF5490T5E"
+			(at 16.51 139.7 0)
+			(hide yes)
+			(show_name no)
+			(do_not_autoplace no)
+			(effects
+				(font
+					(size 1.27 1.27)
+				)
+			)
+		)
+		(pin "2"
+		)
+		(pin "1"
+		)
+		(instances
+			(project "DrunkEarPhoneAdapter"
+				(path "/df940915-8af0-46f9-b18a-23d4684ae671/5c561383-fdd0-44ae-83ac-568aac0f03a9"
+					(reference "R19")
+					(unit 1)
+				)
+			)
+		)
+	)
+	(symbol
 		(lib_id "JLCImport:CL05B102KB5NNNC")
 		(at 36.83 140.97 90)
@@
 					(unit 1)
 				)
-			)
-		)
-	)
-	(symbol
-		(lib_id "JLCImport:0603WAJ0511T5E")
-		(at 137.16 138.43 90)
-		(unit 1)
-		(body_style 1)
-		(exclude_from_sim no)
-		(in_bom yes)
-		(on_board yes)
-		(in_pos_files yes)
-		(dnp no)
-		(fields_autoplaced yes)
-		(property "Reference" "R20"
-			(at 139.7 137.1599 90)
-			(show_name no)
-			(do_not_autoplace no)
-			(effects
-				(font
-					(size 1.27 1.27)
-				)
-				(justify right)
-			)
-		)
-		(property "Value" "510Ω"
-			(at 139.7 139.6999 90)
-			(show_name no)
-			(do_not_autoplace no)
-			(effects
-				(font
-					(size 1.27 1.27)
-				)
-				(justify right)
-			)
-		)
-		(property "Footprint" "Resistor_SMD:R_0603_1608Metric"
-			(at 137.16 138.43 0)
-			(hide yes)
-			(show_name no)
-			(do_not_autoplace no)
-			(effects
-				(font
-					(size 1.27 1.27)
-				)
-			)
-		)
-		(property "Datasheet" "https://www.lcsc.com/datasheet/lcsc_datasheet_2205311845_UNI-ROYAL-Uniroyal-Elec-0603WAJ0511T5E_C25245.pdf"
-			(at 137.16 138.43 0)
-			(hide yes)
-			(show_name no)
-			(do_not_autoplace no)
-			(effects
-				(font
-					(size 1.27 1.27)
-				)
-			)
-		)
-		(property "Description" "-55℃~+155℃ 100mW 510Ω 75V Thick Film Resistor ±100ppm/℃ ±5% 0603 Chip Resistor - Surface Mount ROHS"
-			(at 137.16 138.43 0)
-			(hide yes)
-			(show_name no)
-			(do_not_autoplace no)
-			(effects
-				(font
-					(size 1.27 1.27)
-				)
-			)
-		)
-		(property "LCSC" "C25245"
-			(at 137.16 138.43 0)
-			(hide yes)
-			(show_name no)
-			(do_not_autoplace no)
-			(effects
-				(font
-					(size 1.27 1.27)
-				)
-			)
-		)
-		(property "Manufacturer" "UNI-ROYAL(Uniroyal Elec)"
-			(at 137.16 138.43 0)
-			(hide yes)
-			(show_name no)
-			(do_not_autoplace no)
-			(effects
-				(font
-					(size 1.27 1.27)
-				)
-			)
-		)
-		(property "Manufacturer Part" "0603WAJ0511T5E"
-			(at 137.16 138.43 0)
-			(hide yes)
-			(show_name no)
-			(do_not_autoplace no)
-			(effects
-				(font
-					(size 1.27 1.27)
-				)
-			)
-		)
-		(pin "2"
-		)
-		(pin "1"
-		)
-		(instances
-			(project "DrunkEarPhoneAdapter"
-				(path "/df940915-8af0-46f9-b18a-23d4684ae671/5c561383-fdd0-44ae-83ac-568aac0f03a9"
-					(reference "R20")
-					(unit 1)
-				)

Commit message: Replace parts
Parts:
- removed C44, C74, C84: 100nF 16V X7R, JLCImport:CL05B104KO5NNNC, symbol JLCImport:CL05B104KO5NNNC
- removed C70, C71, C72, C73: 330pF 50V, Capacitor_SMD:C_0402_1005Metric, symbol JLCImport:CL05C331JB5NNNC
- removed C80, C81, C82, C83: 1nF 50V X7R, Capacitor_SMD:C_0402_1005Metric, symbol JLCImport:CL05B102KB5NNNC
- removed C87, C88: 100nF 50V X7R, Capacitor_SMD:C_0402_1005Metric, symbol JLCImport:CC0402KRX7R9BB104
- removed R23, R30: 0Ω, Resistor_SMD:R_0402_1005Metric, symbol JLCImport:RC0402FR-070RL
- removed R40, R41: 10kΩ 0603, Resistor_SMD:R_0603_1608Metric, symbol JLCImport:RC0603FR-0710KL
- added C1, C19, C20, C21, C22: 1nF 50V, Capacitor_SMD:C_0402_1005Metric, symbol JLCImport:0402B102K500NT
- added C23: 4.7uF 16V, Capacitor_SMD:C_0603_1608Metric, symbol JLCImport:CL10A475KO8NNNC
- added C28, C29, C30, C33: 330pF 50V, Capacitor_SMD:C_0603_1608Metric, symbol JLCImport:CL10C331JB8NNNC
- added C74, C78, C84, C87, C88: 100nF 50V, Capacitor_SMD:C_0402_1005Metric, symbol JLCImport:CL05B104KB54PNC
- added R16, R9: 1kΩ, Resistor_SMD:R_0402_1005Metric, symbol JLCImport:0402WGF1001TCE
- added R30, R35: 10kΩ, Resistor_SMD:R_0603_1608Metric, symbol JLCImport:0603WAF1002T5E
Connections:
- net +3V3_D: now also C74.2, C78.2, C84.2
- net ADC_CHR_IANA: now also C21.2, R16.1
- net ADC_CHR_VBUS: now also C22.2
- net ADC_PHONE_IANA: now also C19.2, R9.1
- net ADC_PHONE_VBUS: now also C20.2
- net GND: now also C19.1, C20.1, C21.1, C22.1, C28.1, C29.1, C30.1, C33.1, C74.1, C78.1, C84.1, C87.1, C88.2
- net USB_CHR_CC1: now also C28.2
- net USB_CHR_CC2: now also C29.2
- net USB_CHR_VBUS: now also R35.2
- net USB_PHONE_CC1: now also C30.2
- net USB_PHONE_CC2: now also C33.2
- net USB_PHONE_VBUS: now also R30.2
- net VSENSE_CHR: now also R35.1
- net VSENSE_PHONE: now also R30.1
- net at U5.4 (IANA): now also R16.2
- net at U4.14 (CBIAS): now also C87.2
- net at U5.14 (CBIAS): now also C88.1
- net at U4.4 (IANA): now also R9.2
