File: hardware/d1/dac.kicad_sch (KiCad schematic)
At the start: 48 parts, among them U1 CS43131-CNZR, U14 BLM15PX601SN1D, U17 SN74LVC1G32DBVR, U18 TPS22917DBVR, U19 TPS22917DBVR, U20 SN74AVC4T774RSVR, U21 TCA9406DCUR, X1 22.5792MHz, X3 24.576MHz

Commit message: Fixes
Parts:
- removed C16: 4.7uF 10V X5R, JLCImport:CL05A475MP5NRNC, symbol JLCImport:CL05A475MP5NRNC
- removed C31, C32: 2.2uF 16V X5R, JLCImport:CL05A225KO5NQNC, symbol JLCImport:CL05A225KO5NQNC
- added C2: 4.7uF 10V X5R, Capacitor_SMD:C_0603_1608Metric, symbol JLCImport:CL10A475KP8NNNC
- added C31, C32: 2.2uF 50V X7R, JLCImport:CC0805KKX7R9BB225, symbol JLCImport:CC0805KKX7R9BB225
Connections:
- net GND: now also C2.1, C31.2, C32.2
- net VCP_FILT+: now also C31.1
- net VCP_FILT-: now also C32.1
- net at C21.2, U1.26 (VP), U14.2: now also C2.2
- net JACK_RING_2 renamed HPREFA
- net HPREFA: no longer U1.17 (HPREFB)
- new net HPREFB: U1.17 (HPREFB)
Other:
- note removed: "Need to be two separate connections"

Commit message: Fix Caps
Parts:
- added C85: 1uF 25V X5R, JLCImport:CL05A105KA5NQNC, symbol JLCImport:CL05A105KA5NQNC
Connections:
- net GND: now also C85.2
- net at C22.1, C24.1, L3.2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: now also C85.1
Other:
- moved on the sheet: C24
Changed lines of the file:
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@@
 	)
 	(junction
+		(at 127 152.4)
+		(diameter 0)
+		(color 0 0 0 0)
+	)
+	(junction
 		(at 129.54 129.54)
 		(diameter 0)
@@
 	)
 	(junction
-		(at 124.46 152.4)
+		(at 121.92 152.4)
 		(diameter 0)
 		(color 0 0 0 0)
@@
 	)
 	(junction
+		(at 127 140.97)
+		(diameter 0)
+		(color 0 0 0 0)
+	)
+	(junction
 		(at 102.87 134.62)
 		(diameter 0)
@@
 	(wire
 		(pts
+			(xy 127 152.4) (xy 132.08 152.4)
+		)
+		(stroke
+			(width 0)
+			(type default)
+		)
+	)
+	(wire
+		(pts
 			(xy 135.89 76.2) (xy 135.89 91.44)
 		)
@@
 	(wire
 		(pts
-			(xy 124.46 140.97) (xy 129.54 140.97)
+			(xy 121.92 140.97) (xy 127 140.97)
 		)
 		(stroke
@@
 	(wire
 		(pts
+			(xy 127 140.97) (xy 129.54 140.97)
+		)
+		(stroke
+			(width 0)
+			(type default)
+		)
+	)
+	(wire
+		(pts
 			(xy 227.33 152.4) (xy 214.63 152.4)
 		)
@@
 	(wire
 		(pts
-			(xy 124.46 152.4) (xy 132.08 152.4)
-		)
-		(stroke
-			(width 0)
-			(type default)
-		)
-	)
-	(wire
-		(pts
 			(xy 116.84 138.43) (xy 116.84 142.24)
 		)
@@
 	(wire
 		(pts
-			(xy 116.84 152.4) (xy 124.46 152.4)
+			(xy 116.84 152.4) (xy 127 152.4)
 		)
 		(stroke
@@
 	(wire
 		(pts
-			(xy 124.46 142.24) (xy 124.46 140.97)
+			(xy 121.92 142.24) (xy 121.92 140.97)
 		)
 		(stroke
@@
 	(wire
 		(pts
+			(xy 127 140.97) (xy 127 142.24)
+		)
+		(stroke
+			(width 0)
+			(type default)
+		)
+	)
+	(wire
+		(pts
 			(xy 71.12 49.53) (xy 71.12 43.18)
 		)
@@
 	(symbol
 		(lib_id "JLCImport:CL05B104KO5NNNC")
-		(at 124.46 147.32 270)
+		(at 121.92 147.32 270)
 		(unit 1)
 		(body_style 1)
@@
 		(dnp no)
 		(property "Reference" "C24"
-			(at 119.888 145.542 90)
+			(at 117.348 145.542 90)
 			(show_name no)
 			(do_not_autoplace no)
@@
 		)
 		(property "Value" "100nF 16V X7R"
-			(at 124.46 153.924 0)
+			(at 121.92 153.924 0)
 			(show_name no)
 			(do_not_autoplace no)
@@
 		)
 		(property "Footprint" "JLCImport:CL05B104KO5NNNC"
-			(at 124.46 147.32 0)
+			(at 121.92 147.32 0)
 			(hide yes)
 			(show_name no)
@@
 		)
 		(property "Datasheet" "https://www.lcsc.com/datasheet/lcsc_datasheet_2304140030_Samsung-Electro-Mechanics-CL05B104KO5NNNC_C1525.pdf"
-			(at 124.46 147.32 0)
+			(at 121.92 147.32 0)
 			(hide yes)
 			(show_name no)
@@
 		)
 		(property "Description" "100nF 16V X7R ±10% 0402 Multilayer Ceramic Capacitors MLCC - SMD/SMT ROHS"
-			(at 124.46 147.32 0)
+			(at 121.92 147.32 0)
 			(hide yes)
 			(show_name no)
@@
 		)
 		(property "LCSC" "C1525"
-			(at 124.46 147.32 0)
+			(at 121.92 147.32 0)
 			(hide yes)
 			(show_name no)
@@
 		)
 		(property "Manufacturer" "Samsung Electro-Mechanics"
-			(at 124.46 147.32 0)
+			(at 121.92 147.32 0)
 			(hide yes)
 			(show_name no)
@@
 		)
 		(property "Manufacturer Part" "CL05B104KO5NNNC"
-			(at 124.46 147.32 0)
+			(at 121.92 147.32 0)
 			(hide yes)
 			(show_name no)
@@
 		(dnp no)
 		(property "Reference" "C23"
-			(at 131.318 145.288 90)
+			(at 131.064 145.288 90)
 			(show_name no)
 			(do_not_autoplace no)
@@
 					(unit 1)
 				)
+			)
+		)
+	)
+	(symbol
+		(lib_id "JLCImport:CL05A105KA5NQNC")
+		(at 127 147.32 270)
+		(unit 1)
+		(body_style 1)
+		(exclude_from_sim no)
+		(in_bom yes)
+		(on_board yes)
+		(in_pos_files yes)
+		(dnp no)
+		(property "Reference" "C85"
+			(at 126.238 145.288 90)
+			(show_name no)
+			(do_not_autoplace no)
+			(effects
+				(font
+					(size 1.27 1.27)
+				)
+				(justify right)
+			)
+		)
+		(property "Value" "1uF 25V X5R"
+			(at 125.984 166.116 0)
+			(show_name no)
+			(do_not_autoplace no)
+			(effects
+				(font
+					(size 1.27 1.27)
+				)
+				(justify right)
+			)
+		)
+		(property "Footprint" "JLCImport:CL05A105KA5NQNC"
+			(at 127 147.32 0)
+			(hide yes)
+			(show_name no)
+			(do_not_autoplace no)
+			(effects
+				(font
+					(size 1.27 1.27)
+				)
+			)
+		)
+		(property "Datasheet" "https://www.lcsc.com/datasheet/lcsc_datasheet_2304140030_Samsung-Electro-Mechanics-CL05A105KA5NQNC_C52923.pdf"
+			(at 127 147.32 0)
+			(hide yes)
+			(show_name no)
+			(do_not_autoplace no)
+			(effects
+				(font
+					(size 1.27 1.27)
+				)
+			)
+		)
+		(property "Description" "1uF 25V X5R ±10% 0402 Multilayer Ceramic Capacitors MLCC - SMD/SMT ROHS"
+			(at 127 147.32 0)
+			(hide yes)
+			(show_name no)
+			(do_not_autoplace no)
+			(effects
+				(font
+					(size 1.27 1.27)
+				)
+			)
+		)
+		(property "LCSC" "C52923"
+			(at 127 147.32 0)
+			(hide yes)
+			(show_name no)
+			(do_not_autoplace no)
+			(effects
+				(font
+					(size 1.27 1.27)
+				)
+			)
+		)
+		(property "Manufacturer" "Samsung Electro-Mechanics"
+			(at 127 147.32 0)
+			(hide yes)
+			(show_name no)
+			(do_not_autoplace no)
+			(effects
+				(font
+					(size 1.27 1.27)
+				)
+			)
+		)
+		(property "Manufacturer Part" "CL05A105KA5NQNC"
+			(at 127 147.32 0)
+			(hide yes)
+			(show_name no)
+			(do_not_autoplace no)
+			(effects
+				(font
+					(size 1.27 1.27)
+				)
+			)
+		)
+		(pin "2"
+		)
+		(pin "1"
+		)
+		(instances
+			(project "DrunkEarPhoneAdapter"
+				(path "/df940915-8af0-46f9-b18a-23d4684ae671/95ba76fd-cd0d-4fc7-9d47-f5665dc7e9c9"
+					(reference "C85")
+					(unit 1)
+				)

Commit message: Replace parts
Parts:
- removed C19, C21, C22, C23, C24, C77, C78, C79, C89, C90, C91, C92: 100nF 16V X7R, JLCImport:CL05B104KO5NNNC, symbol JLCImport:CL05B104KO5NNNC
- removed C2: 4.7uF 10V X5R, Capacitor_SMD:C_0603_1608Metric, symbol JLCImport:CL10A475KP8NNNC
- removed C25, C28, C29, C30, C33, C34: 2.2uF 16V X5R, JLCImport:CL05A225KO5NQNC, symbol JLCImport:CL05A225KO5NQNC
- removed C26, C27: 15uF 35V X5R, JLCImport:C2012X5R1V156MT000E, symbol JLCImport:C2012X5R1V156MT000E
- removed R16, R38, R9: 33Ω, Resistor_SMD:R_0402_1005Metric, symbol JLCImport:RC0402FR-0733RL
- removed R35: 1kΩ, Resistor_SMD:R_0402_1005Metric, symbol JLCImport:RC0402FR-071KL
- added C101, C102, C103, C104, C53, C55, C77, C89, C90, C91, C92, C98: 100nF 50V, Capacitor_SMD:C_0402_1005Metric, symbol JLCImport:CL05B104KB54PNC
- added C13, C16, C2, C25, C3, C7: 2.2uF 16V, Capacitor_SMD:C_0603_1608Metric, symbol JLCImport:CL10A225KO8NNNC
- added C24: 4.7uF 16V, Capacitor_SMD:C_0603_1608Metric, symbol JLCImport:CL10A475KO8NNNC
- added C26, C27: 22uF 25V X5R, JLCImport:CL21A226MAQNNNE, symbol JLCImport:CL21A226MAQNNNE
- added R23: 1kΩ, Resistor_SMD:R_0402_1005Metric, symbol JLCImport:0402WGF1001TCE
- added R27, R38, R43, R44: 33Ω, Resistor_SMD:R_0402_1005Metric, symbol JLCImport:0402WGF330JTCE
Connections:
- net +1V8_A: now also C103.2, C2.2, C26.2
- net +1V8_CP: now also C13.1
- net +1V8_D: now also C89.1, C92.1
- net +3V3_D: now also C90.2, C91.1
- net -VA: now also C27.2, C3.1
- net CLKOUT: now also R43.2
- net FILT+: now also C26.1
- net FILT-: now also C27.1
- net FLYC_VCP: now also C16.2, C25.1
- net FLYN_VA: now also C7.1
- net FLYN_VCP: now also C25.2
- net FLYP_VA: now also C7.2
- net FLYP_VCP: now also C16.1
- net GND: now also C101.1, C102.1, C103.1, C104.1, C13.2, C2.1, C24.1, C3.2, C53.1, C55.1, C77.2, C89.2, C90.1, C91.2, C92.2, C98.2
- net I2S_CK: now also R38.2
- net JACK_TIP_DETECT: now also R23.2
- net at C93.1, C94.1, L1.2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: now also C53.2, C55.2
- net at C85.1, L3.2, U1.31 (VL)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: now also C101.2, C102.2
- net at U1.26 (VP), U14.2: now also C104.2, C24.2
- net at U1.22 (HP_DETECT): now also R23.1
- net at U17.4 (Y): now also R44.1
- net at C76.2, U19.5 (QOD), U19.6 (VOUT)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: now also C77.1
- net at U20.12 (B1): now also R38.1
- net at C17.2, U18.5 (QOD), U18.6 (VOUT)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: now also C98.1
- net at U20.10 (B3): now also R43.1
- net at U1.37 (XTI/MCLK): now also R44.2
Other:
- moved on the sheet: C94

Commit message: Fix parts
Parts:
- removed R27: 33Ω, Resistor_SMD:R_0402_1005Metric, symbol JLCImport:0402WGF330JTCE
Changed lines of the file:
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@@
-	)
-	(symbol
-		(lib_id "JLCImport:0402WGF330JTCE")
-		(at 118.11 22.86 0)
-		(unit 1)
-		(body_style 1)
-		(exclude_from_sim no)
-		(in_bom yes)
-		(on_board yes)
-		(in_pos_files yes)
-		(dnp no)
-		(fields_autoplaced yes)
-		(property "Reference" "R27"
-			(at 118.11 16.51 0)
-			(show_name no)
-			(do_not_autoplace no)
-			(effects
-				(font
-					(size 1.27 1.27)
-				)
-			)
-		)
-		(property "Value" "33Ω"
-			(at 118.11 19.05 0)
-			(show_name no)
-			(do_not_autoplace no)
-			(effects
-				(font
-					(size 1.27 1.27)
-				)
-			)
-		)
-		(property "Footprint" "Resistor_SMD:R_0402_1005Metric"
-			(at 118.11 22.86 0)
-			(hide yes)
-			(show_name no)
-			(do_not_autoplace no)
-			(effects
-				(font
-					(size 1.27 1.27)
-				)
-			)
-		)
-		(property "Datasheet" "https://www.lcsc.com/datasheet/lcsc_datasheet_2205311900_UNI-ROYAL-Uniroyal-Elec-0402WGF330JTCE_C25105.pdf"
-			(at 118.11 22.86 0)
-			(hide yes)
-			(show_name no)
-			(do_not_autoplace no)
-			(effects
-				(font
-					(size 1.27 1.27)
-				)
-			)
-		)
-		(property "Description" "-55℃~+155℃ 33Ω 50V 62.5mW Thick Film Resistor ±1% ±100ppm/℃ 0402 Chip Resistor - Surface Mount ROHS"
-			(at 118.11 22.86 0)
-			(hide yes)
-			(show_name no)
-			(do_not_autoplace no)
-			(effects
-				(font
-					(size 1.27 1.27)
-				)
-			)
-		)
-		(property "LCSC" "C25105"
-			(at 118.11 22.86 0)
-			(hide yes)
-			(show_name no)
-			(do_not_autoplace no)
-			(effects
-				(font
-					(size 1.27 1.27)
-				)
-			)
-		)
-		(property "Manufacturer" "UNI-ROYAL(Uniroyal Elec)"
-			(at 118.11 22.86 0)
-			(hide yes)
-			(show_name no)
-			(do_not_autoplace no)
-			(effects
-				(font
-					(size 1.27 1.27)
-				)
-			)
-		)
-		(property "Manufacturer Part" "0402WGF330JTCE"
-			(at 118.11 22.86 0)
-			(hide yes)
-			(show_name no)
-			(do_not_autoplace no)
-			(effects
-				(font
-					(size 1.27 1.27)
-				)
-			)
-		)
-		(pin "2"
-		)
-		(pin "1"
-		)
-		(instances
-			(project "DrunkEarPhoneAdapter"
-				(path "/df940915-8af0-46f9-b18a-23d4684ae671/95ba76fd-cd0d-4fc7-9d47-f5665dc7e9c9"
-					(reference "R27")
-					(unit 1)
-				)
-			)
-		)
 	)
 	(symbol

Commit message: Fix routes
Parts:
- added C107: 100nF 50V, Capacitor_SMD:C_0402_1005Metric, symbol JLCImport:CL05B104KB54PNC
Connections:
- net GND: now also C107.2
- net at C53.2, C55.2, C93.1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: now also C107.1
Changed lines of the file:
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@@
 	)
 	(junction
+		(at 110.49 45.72)
+		(diameter 0)
+		(color 0 0 0 0)
+	)
+	(junction
 		(at 76.2 60.96)
 		(diameter 0)
@@
 	(wire
 		(pts
-			(xy 110.49 40.64) (xy 110.49 67.31)
+			(xy 110.49 40.64) (xy 110.49 45.72)
 		)
 		(stroke
@@
 	(wire
 		(pts
+			(xy 110.49 45.72) (xy 110.49 67.31)
+		)
+		(stroke
+			(width 0)
+			(type default)
+		)
+	)
+	(wire
+		(pts
 			(xy 76.2 43.18) (xy 96.52 43.18)
 		)
@@
 	)
 	(symbol
+		(lib_id "JLCImport:CL05B104KB54PNC")
+		(at 115.57 45.72 0)
+		(unit 1)
+		(body_style 1)
+		(exclude_from_sim no)
+		(in_bom yes)
+		(on_board yes)
+		(in_pos_files yes)
+		(dnp no)
+		(property "Reference" "C107"
+			(at 112.776 44.45 0)
+			(show_name no)
+			(do_not_autoplace no)
+			(effects
+				(font
+					(size 1.27 1.27)
+				)
+			)
+		)
+		(property "Value" "100nF 50V"
+			(at 115.57 49.53 0)
+			(show_name no)
+			(do_not_autoplace no)
+			(effects
+				(font
+					(size 1.27 1.27)
+				)
+			)
+		)
+		(property "Footprint" "Capacitor_SMD:C_0402_1005Metric"
+			(at 115.57 45.72 0)
+			(hide yes)
+			(show_name no)
+			(do_not_autoplace no)
+			(effects
+				(font
+					(size 1.27 1.27)
+				)
+			)
+		)
+		(property "Datasheet" "https://www.lcsc.com/datasheet/lcsc_datasheet_2304140030_Samsung-Electro-Mechanics-CL05B104KB54PNC_C307331.pdf"
+			(at 115.57 45.72 0)
+			(hide yes)
+			(show_name no)
+			(do_not_autoplace no)
+			(effects
+				(font
+					(size 1.27 1.27)
+				)
+			)
+		)
+		(property "Description" "100nF 50V X7R ±10% 0402 Multilayer Ceramic Capacitors MLCC - SMD/SMT ROHS"
+			(at 115.57 45.72 0)
+			(hide yes)
+			(show_name no)
+			(do_not_autoplace no)
+			(effects
+				(font
+					(size 1.27 1.27)
+				)
+			)
+		)
+		(property "LCSC" "C307331"
+			(at 115.57 45.72 0)
+			(hide yes)
+			(show_name no)
+			(do_not_autoplace no)
+			(effects
+				(font
+					(size 1.27 1.27)
+				)
+			)
+		)
+		(property "Manufacturer" "Samsung Electro-Mechanics"
+			(at 115.57 45.72 0)
+			(hide yes)
+			(show_name no)
+			(do_not_autoplace no)
+			(effects
+				(font
+					(size 1.27 1.27)
+				)
+			)
+		)
+		(property "Manufacturer Part" "CL05B104KB54PNC"
+			(at 115.57 45.72 0)
+			(hide yes)
+			(show_name no)
+			(do_not_autoplace no)
+			(effects
+				(font
+					(size 1.27 1.27)
+				)
+			)
+		)
+		(pin "2"
+		)
+		(pin "1"
+		)
+		(instances
+			(project "DrunkEarPhoneAdapter"
+				(path "/df940915-8af0-46f9-b18a-23d4684ae671/95ba76fd-cd0d-4fc7-9d47-f5665dc7e9c9"
+					(reference "C107")
+					(unit 1)
+				)
+			)
+		)
+	)
+	(symbol
 		(lib_id "JLCImport:CC0805KKX7R9BB225")
 		(at 222.25 21.59 0)
@@
 					(unit 1)
 				)
+			)
+		)
+	)
+	(symbol
+		(lib_id "power:GND")
+		(at 120.65 45.72 90)
+		(unit 1)
+		(body_style 1)
+		(exclude_from_sim no)
+		(in_bom yes)
+		(on_board yes)
+		(in_pos_files yes)
+		(dnp no)
+		(fields_autoplaced yes)
+		(property "Reference" "#PWR093"
+			(at 127 45.72 0)
+			(hide yes)
+			(show_name no)
+			(do_not_autoplace no)
+			(effects
+				(font
+					(size 1.27 1.27)
+				)
+			)
+		)
+		(property "Value" "GND"
+			(at 124.46 45.7199 90)
+			(show_name no)
+			(do_not_autoplace no)
+			(effects
+				(font
+					(size 1.27 1.27)
+				)
+				(justify right)
+			)
+		)
+		(property "Footprint" ""
+			(at 120.65 45.72 0)
+			(hide yes)
+			(show_name no)
+			(do_not_autoplace no)
+			(effects
+				(font
+					(size 1.27 1.27)
+				)
+			)
+		)
+		(property "Datasheet" ""
+			(at 120.65 45.72 0)
+			(hide yes)
+			(show_name no)
+			(do_not_autoplace no)
+			(effects
+				(font
+					(size 1.27 1.27)
+				)
+			)
+		)
+		(property "Description" "Power symbol creates a global label with name \"GND\" , ground"
+			(at 120.65 45.72 0)
+			(hide yes)
+			(show_name no)
+			(do_not_autoplace no)
+			(effects
+				(font
+					(size 1.27 1.27)
+				)
+			)
+		)
+		(pin "1"
+		)
+		(instances
+			(project "DrunkEarPhoneAdapter"
+				(path "/df940915-8af0-46f9-b18a-23d4684ae671/95ba76fd-cd0d-4fc7-9d47-f5665dc7e9c9"
+					(reference "#PWR093")
+					(unit 1)
+				)
