File: hardware/d1/mcu.kicad_sch (KiCad schematic)
At the start: 24 parts, among them J3 SWD, J4 UART, Q3 DMG1012T-7, U2 STM32G0B1VCT6

Commit message: Fixes
Parts:
- removed C53, C55: 4.7uF 10V X5R, JLCImport:CL05A475MP5NRNC, symbol JLCImport:CL05A475MP5NRNC
- added C16, C7: 4.7uF 10V X5R, Capacitor_SMD:C_0603_1608Metric, symbol JLCImport:CL10A475KP8NNNC
- added R43: 100kΩ, JLCImport:0402WGF1003TCE, symbol JLCImport:0402WGF1003TCE
- added SW1: SSSS811101, JLCImport:SSSS811101, symbol JLCImport:SSSS811101
Connections:
- net +3V3_D: now also C16.2, C7.2, SW1.3
- net GND: now also C16.1, C7.1, R43.2, SW1.1, SW1.4, SW1.5, SW1.6, SW1.7
- net USB_DIR: now reaches U2.59 (PD8)
- net USB_DIR_SW: now reaches U2.60 (PD9)
- net USB_DIR_SW: now also R43.1, SW1.2
Other:
- moved on the sheet: Q3, R39

Commit message: Fixes
Parts:
- removed R43: 100kΩ, JLCImport:0402WGF1003TCE, symbol JLCImport:0402WGF1003TCE
- added R26: 47kΩ, Resistor_SMD:R_0402_1005Metric, symbol JLCImport:0402WGF4702TCE
Connections:
- net GND: now also R26.2; no longer SW1.1
- net USB_DIR_SW: now also R26.1
- no-connect marks 4 -> 5
Changed lines of the file:
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@@
 	)
 	(junction
-		(at 248.92 115.57)
-		(diameter 0)
-		(color 0 0 0 0)
-	)
-	(junction
 		(at 63.5 45.72)
 		(diameter 0)
@@
 	)
 	(junction
+		(at 248.92 115.57)
+		(diameter 0)
+		(color 0 0 0 0)
+	)
+	(junction
 		(at 33.02 86.36)
 		(diameter 0)
@@
 	)
 	(junction
-		(at 238.76 120.65)
-		(diameter 0)
-		(color 0 0 0 0)
-	)
-	(junction
 		(at 257.81 36.83)
 		(diameter 0)
@@
 	)
 	(no_connect
+		(at 246.38 120.65)
+	)
+	(no_connect
 		(at 137.16 78.74)
 	)
@@
 	(wire
 		(pts
+			(xy 259.08 120.65) (xy 254 120.65)
+		)
+		(stroke
+			(width 0)
+			(type default)
+		)
+	)
+	(wire
+		(pts
 			(xy 195.58 66.04) (xy 199.39 66.04)
 		)
@@
 	(wire
 		(pts
-			(xy 248.92 115.57) (xy 248.92 120.65)
+			(xy 248.92 109.22) (xy 248.92 115.57)
 		)
 		(stroke
@@
 	(wire
 		(pts
-			(xy 35.56 181.61) (xy 39.37 181.61)
+			(xy 248.92 115.57) (xy 248.92 120.65)
 		)
 		(stroke
@@
 	(wire
 		(pts
-			(xy 35.56 161.29) (xy 39.37 161.29)
+			(xy 35.56 181.61) (xy 39.37 181.61)
 		)
 		(stroke
@@
 	(wire
 		(pts
-			(xy 147.32 71.12) (xy 137.16 71.12)
+			(xy 35.56 161.29) (xy 39.37 161.29)
 		)
 		(stroke
@@
 	(wire
 		(pts
-			(xy 257.81 26.67) (xy 251.46 26.67)
+			(xy 147.32 71.12) (xy 137.16 71.12)
 		)
 		(stroke
@@
 	(wire
 		(pts
-			(xy 251.46 41.91) (xy 257.81 41.91)
+			(xy 257.81 26.67) (xy 251.46 26.67)
 		)
 		(stroke
@@
 	(wire
 		(pts
-			(xy 68.58 45.72) (xy 63.5 45.72)
+			(xy 251.46 41.91) (xy 257.81 41.91)
 		)
 		(stroke
@@
 	(wire
 		(pts
-			(xy 68.58 71.12) (xy 83.82 71.12)
+			(xy 68.58 45.72) (xy 63.5 45.72)
 		)
 		(stroke
@@
 	(wire
 		(pts
-			(xy 29.21 45.72) (xy 35.56 45.72)
+			(xy 68.58 71.12) (xy 83.82 71.12)
 		)
 		(stroke
@@
 	(wire
 		(pts
-			(xy 238.76 120.65) (xy 246.38 120.65)
+			(xy 29.21 45.72) (xy 35.56 45.72)
 		)
 		(stroke
@@
 	(wire
 		(pts
-			(xy 248.92 109.22) (xy 248.92 115.57)
-		)
-		(stroke
-			(width 0)
-			(type default)
-		)
-	)
-	(wire
-		(pts
 			(xy 81.28 25.4) (xy 49.53 25.4)
 		)
@@
 	)
 	(symbol
-		(lib_id "JLCImport:CL05B104KO5NNNC")
-		(at 201.93 151.13 270)
+		(lib_id "JLCImport:0402WGF4702TCE")
+		(at 243.84 115.57 180)
 		(unit 1)
 		(body_style 1)
@@
 		(in_pos_files yes)
 		(dnp no)
-		(property "Reference" "C50"
-			(at 199.136 152.908 0)
+		(property "Reference" "R26"
+			(at 243.84 117.856 0)
 			(show_name no)
 			(do_not_autoplace no)
@@
 					(size 1.27 1.27)
 				)
-				(justify left)
 			)
 		)
-		(property "Value" "100nF 16V X7R"
-			(at 204.724 152.908 0)
+		(property "Value" "47kΩ"
+			(at 243.84 113.538 0)
 			(show_name no)
 			(do_not_autoplace no)
@@
 					(size 1.27 1.27)
 				)
-				(justify left)
 			)
 		)
-		(property "Footprint" "JLCImport:CL05B104KO5NNNC"
-			(at 201.93 151.13 0)
+		(property "Footprint" "Resistor_SMD:R_0402_1005Metric"
+			(at 243.84 115.57 0)
 			(hide yes)
 			(show_name no)
@@
 			)
 		)
-		(property "Datasheet" "https://www.lcsc.com/datasheet/lcsc_datasheet_2304140030_Samsung-Electro-Mechanics-CL05B104KO5NNNC_C1525.pdf"
-			(at 201.93 151.13 0)
+		(property "Datasheet" "https://www.lcsc.com/datasheet/lcsc_datasheet_2206010100_UNI-ROYAL-Uniroyal-Elec-0402WGF4702TCE_C25792.pdf"
+			(at 243.84 115.57 0)
 			(hide yes)
 			(show_name no)
@@
 			)
 		)
-		(property "Description" "100nF 16V X7R ±10% 0402 Multilayer Ceramic Capacitors MLCC - SMD/SMT ROHS"
-			(at 201.93 151.13 0)
+		(property "Description" "-55℃~+155℃ 47kΩ 50V 62.5mW Thick Film Resistor ±1% ±100ppm/℃ 0402 Chip Resistor - Surface Mount ROHS"
+			(at 243.84 115.57 0)
 			(hide yes)
 			(show_name no)
@@
 			)
 		)
-		(property "LCSC" "C1525"
-			(at 201.93 151.13 0)
+		(property "LCSC" "C25792"
+			(at 243.84 115.57 0)
 			(hide yes)
 			(show_name no)
@@
 			)
 		)
-		(property "Manufacturer" "Samsung Electro-Mechanics"
-			(at 201.93 151.13 0)
+		(property "Manufacturer" "UNI-ROYAL(Uniroyal Elec)"
+			(at 243.84 115.57 0)
 			(hide yes)
 			(show_name no)
@@
 			)
 		)
-		(property "Manufacturer Part" "CL05B104KO5NNNC"
-			(at 201.93 151.13 0)
+		(property "Manufacturer Part" "0402WGF4702TCE"
+			(at 243.84 115.57 0)
 			(hide yes)
 			(show_name no)
@@
 			(project "DrunkEarPhoneAdapter"
 				(path "/df940915-8af0-46f9-b18a-23d4684ae671/c6b936ac-23e1-4f20-8d3d-ded05833abcb"
-					(reference "C50")
+					(reference "R26")
 					(unit 1)
 				)
@@
 	)
 	(symbol
-		(lib_id "JLCImport:0402WGF1003TCE")
-		(at 243.84 115.57 180)
+		(lib_id "JLCImport:CL05B104KO5NNNC")
+		(at 201.93 151.13 270)
 		(unit 1)
 		(body_style 1)
@@
 		(in_pos_files yes)
 		(dnp no)
-		(property "Reference" "R43"
-			(at 244.094 117.856 0)
+		(property "Reference" "C50"
+			(at 199.136 152.908 0)
 			(show_name no)
 			(do_not_autoplace no)
@@
 					(size 1.27 1.27)
 				)
+				(justify left)
 			)
 		)
-		(property "Value" "100kΩ"
-			(at 243.84 113.284 0)
+		(property "Value" "100nF 16V X7R"
+			(at 204.724 152.908 0)
 			(show_name no)
 			(do_not_autoplace no)
@@
 					(size 1.27 1.27)
 				)
+				(justify left)
 			)
 		)
-		(property "Footprint" "JLCImport:0402WGF1003TCE"
-			(at 243.84 115.57 0)
+		(property "Footprint" "JLCImport:CL05B104KO5NNNC"
+			(at 201.93 151.13 0)
 			(hide yes)
 			(show_name no)
@@
 			)
 		)
-		(property "Datasheet" "https://www.lcsc.com/datasheet/lcsc_datasheet_2206010100_UNI-ROYAL-Uniroyal-Elec-0402WGF1003TCE_C25741.pdf"
-			(at 243.84 115.57 0)
+		(property "Datasheet" "https://www.lcsc.com/datasheet/lcsc_datasheet_2304140030_Samsung-Electro-Mechanics-CL05B104KO5NNNC_C1525.pdf"
+			(at 201.93 151.13 0)
 			(hide yes)
 			(show_name no)
@@
 			)
 		)
-		(property "Description" "-55℃~+155℃ 100kΩ 50V 62.5mW Thick Film Resistor ±1% ±100ppm/℃ 0402 Chip Resistor - Surface Mount ROHS"
-			(at 243.84 115.57 0)
+		(property "Description" "100nF 16V X7R ±10% 0402 Multilayer Ceramic Capacitors MLCC - SMD/SMT ROHS"
+			(at 201.93 151.13 0)
 			(hide yes)
 			(show_name no)
@@
 			)
 		)
-		(property "LCSC" "C25741"
-			(at 243.84 115.57 0)
+		(property "LCSC" "C1525"
+			(at 201.93 151.13 0)
 			(hide yes)
 			(show_name no)
@@
 			)
 		)
-		(property "Manufacturer" "UNI-ROYAL(Uniroyal Elec)"
-			(at 243.84 115.57 0)
+		(property "Manufacturer" "Samsung Electro-Mechanics"
+			(at 201.93 151.13 0)
 			(hide yes)
 			(show_name no)
@@
 			)
 		)
-		(property "Manufacturer Part" "0402WGF1003TCE"
-			(at 243.84 115.57 0)
+		(property "Manufacturer Part" "CL05B104KO5NNNC"
+			(at 201.93 151.13 0)
 			(hide yes)
 			(show_name no)
@@
 			(project "DrunkEarPhoneAdapter"
 				(path "/df940915-8af0-46f9-b18a-23d4684ae671/c6b936ac-23e1-4f20-8d3d-ded05833abcb"
-					(reference "R43")
+					(reference "C50")
 					(unit 1)
 				)
@@
 	(symbol
 		(lib_id "power:+3V8")
-		(at 254 120.65 0)
+		(at 259.08 120.65 0)
 		(unit 1)
 		(body_style 1)
@@
 		(fields_autoplaced yes)
 		(property "Reference" "#PWR089"
-			(at 254 124.46 0)
+			(at 259.08 124.46 0)
 			(hide yes)
 			(show_name no)
@@
 		)
 		(property "Value" "+3V3_D"
-			(at 254 115.57 0)
+			(at 259.08 115.57 0)
 			(show_name no)
 			(do_not_autoplace no)
@@
 		)
 		(property "Footprint" ""
-			(at 254 120.65 0)
+			(at 259.08 120.65 0)
 			(hide yes)
 			(show_name no)
@@
 		)
 		(property "Datasheet" ""
-			(at 254 120.65 0)
+			(at 259.08 120.65 0)
 			(hide yes)
 			(show_name no)
@@
 		)
 		(property "Description" "Power symbol creates a global label with name \"+3V8\""
-			(at 254 120.65 0)
+			(at 259.08 120.65 0)
 			(hide yes)
 			(show_name no)

Commit message: Replace parts
Parts:
- removed C16, C7: 4.7uF 10V X5R, Capacitor_SMD:C_0603_1608Metric, symbol JLCImport:CL10A475KP8NNNC
- removed C20, C50, C52, C54, C56, C69: 100nF 16V X7R, JLCImport:CL05B104KO5NNNC, symbol JLCImport:CL05B104KO5NNNC
- added C100, C106, C54, C56, C69, C97: 100nF 50V, Capacitor_SMD:C_0402_1005Metric, symbol JLCImport:CL05B104KB54PNC
- added C37, C39: 4.7uF 16V, Capacitor_SMD:C_0603_1608Metric, symbol JLCImport:CL10A475KO8NNNC
Connections:
- net +3V3_D: now also C106.2, C37.2, C39.2, C54.2, C69.2
- net GND: now also C100.1, C106.1, C37.1, C39.1, C54.1, C56.2, C69.1, C97.1
- net NRST: now also C56.1
- net at C18.1, L4.2, U2.12 (VREF+): now also C100.2, C97.2

Commit message: Trace
Connections:
- no-connect marks 5 -> 54
Changed lines of the file:
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@@
+	)
+	(no_connect
+		(at 137.16 116.84)
+	)
+	(no_connect
+		(at 137.16 162.56)
+	)
+	(no_connect
+		(at 137.16 157.48)
 	)
 	(no_connect
@@
 	)
 	(no_connect
+		(at 137.16 40.64)
+	)
+	(no_connect
+		(at 83.82 147.32)
+	)
+	(no_connect
+		(at 83.82 68.58)
+	)
+	(no_connect
 		(at 246.38 120.65)
+	)
+	(no_connect
+		(at 83.82 78.74)
+	)
+	(no_connect
+		(at 83.82 76.2)
+	)
+	(no_connect
+		(at 83.82 63.5)
+	)
+	(no_connect
+		(at 83.82 104.14)
+	)
+	(no_connect
+		(at 83.82 137.16)
+	)
+	(no_connect
+		(at 137.16 144.78)
+	)
+	(no_connect
+		(at 83.82 81.28)
+	)
+	(no_connect
+		(at 137.16 96.52)
+	)
+	(no_connect
+		(at 83.82 167.64)
 	)
 	(no_connect
@@
 	)
 	(no_connect
+		(at 83.82 144.78)
+	)
+	(no_connect
+		(at 137.16 142.24)
+	)
+	(no_connect
+		(at 137.16 45.72)
+	)
+	(no_connect
+		(at 137.16 73.66)
+	)
+	(no_connect
+		(at 137.16 160.02)
+	)
+	(no_connect
+		(at 137.16 170.18)
+	)
+	(no_connect
+		(at 137.16 124.46)
+	)
+	(no_connect
+		(at 137.16 66.04)
+	)
+	(no_connect
+		(at 137.16 165.1)
+	)
+	(no_connect
+		(at 83.82 58.42)
+	)
+	(no_connect
+		(at 83.82 73.66)
+	)
+	(no_connect
+		(at 83.82 127)
+	)
+	(no_connect
+		(at 83.82 154.94)
+	)
+	(no_connect
 		(at 137.16 76.2)
+	)
+	(no_connect
+		(at 137.16 152.4)
+	)
+	(no_connect
+		(at 137.16 114.3)
+	)
+	(no_connect
+		(at 83.82 142.24)
+	)
+	(no_connect
+		(at 243.84 92.71)
+	)
+	(no_connect
+		(at 137.16 167.64)
+	)
+	(no_connect
+		(at 137.16 119.38)
 	)
 	(no_connect
 		(at 83.82 50.8)
 	)
+	(no_connect
+		(at 137.16 111.76)
+	)
+	(no_connect
+		(at 83.82 139.7)
+	)
+	(no_connect
+		(at 83.82 60.96)
+	)
+	(no_connect
+		(at 137.16 63.5)
+	)
+	(no_connect
+		(at 83.82 162.56)
+	)
+	(no_connect
+		(at 137.16 121.92)
+	)
+	(no_connect
+		(at 137.16 50.8)
+	)
+	(no_connect
+		(at 137.16 43.18)
+	)
+	(no_connect
+		(at 137.16 147.32)
+	)
+	(no_connect
+		(at 137.16 68.58)
+	)
+	(no_connect
+		(at 137.16 149.86)
+	)
+	(no_connect
+		(at 137.16 154.94)
+	)
+	(no_connect
+		(at 83.82 55.88)
+	)
+	(no_connect
+		(at 137.16 53.34)
+	)
+	(no_connect
+		(at 83.82 66.04)
+	)
 	(wire

Commit message: Almost done tracing
Connections:
- net UCPD1_FRSTX2: no longer names the net of U2.53 (PB14)
- net UCPD2_FRSTX1: no longer names the net of U2.51 (PB12)
- net UCPD2_FRSTX2: no longer names the net of U2.76 (PC8)
- no-connect marks 54 -> 57
Changed lines of the file:
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@@
+	)
+	(no_connect
+		(at 83.82 170.18)
 	)
 	(no_connect
@@
 	)
 	(no_connect
+		(at 83.82 165.1)
+	)
+	(no_connect
 		(at 137.16 170.18)
 	)
@@
 	)
 	(no_connect
+		(at 137.16 60.96)
+	)
+	(no_connect
 		(at 83.82 162.56)
 	)
@@
 	(wire
 		(pts
-			(xy 77.47 170.18) (xy 83.82 170.18)
-		)
-		(stroke
-			(width 0)
-			(type default)
-		)
-	)
-	(wire
-		(pts
 			(xy 77.47 124.46) (xy 83.82 124.46)
 		)
@@
 	(wire
 		(pts
-			(xy 147.32 60.96) (xy 137.16 60.96)
-		)
-		(stroke
-			(width 0)
-			(type default)
-		)
-	)
-	(wire
-		(pts
 			(xy 187.96 44.45) (xy 194.31 44.45)
 		)
@@
 			(width 0)
 			(type default)
-		)
-	)
-	(wire
-		(pts
-			(xy 77.47 165.1) (xy 83.82 165.1)
-		)
-		(stroke
-			(width 0)
-			(type default)
-		)
-	)
-	(label "UCPD2_FRSTX1"
-		(at 77.47 165.1 180)
-		(effects
-			(font
-				(size 1.27 1.27)
-			)
-			(justify right bottom)
 		)
 	)
@@
 		)
 	)
-	(label "UCPD1_FRSTX2"
-		(at 77.47 170.18 180)
-		(effects
-			(font
-				(size 1.27 1.27)
-			)
-			(justify right bottom)
-		)
-	)
 	(label "UCPD1_DBCC1"
 		(at 241.3 26.67 180)
@@
 		(effects
 			(font
-				(size 1.27 1.27)
-			)
-			(justify left bottom)
-		)
-	)
-	(label "UCPD2_FRSTX2"
-		(at 147.32 60.96 0)
-		(effects
-			(font

Commit message: Fix routes
Parts:
- added C108: 100nF 50V, Capacitor_SMD:C_0402_1005Metric, symbol JLCImport:CL05B104KB54PNC
Connections:
- net GND: now also C108.1
- net at C100.2, C18.1, C97.2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: now also C108.2
Changed lines of the file:
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@@
 	)
 	(junction
+		(at 29.21 35.56)
+		(diameter 0)
+		(color 0 0 0 0)
+	)
+	(junction
 		(at 255.27 134.62)
 		(diameter 0)
@@
 	)
 	(junction
+		(at 29.21 45.72)
+		(diameter 0)
+		(color 0 0 0 0)
+	)
+	(junction
 		(at 111.76 19.05)
 		(diameter 0)
@@
 	(wire
 		(pts
+			(xy 20.32 35.56) (xy 29.21 35.56)
+		)
+		(stroke
+			(width 0)
+			(type default)
+		)
+	)
+	(wire
+		(pts
 			(xy 257.81 41.91) (xy 257.81 36.83)
 		)
@@
 	(wire
 		(pts
+			(xy 20.32 45.72) (xy 29.21 45.72)
+		)
+		(stroke
+			(width 0)
+			(type default)
+		)
+	)
+	(wire
+		(pts
 			(xy 257.81 26.67) (xy 251.46 26.67)
 		)
@@
 					(unit 1)
 				)
+			)
+		)
+	)
+	(symbol
+		(lib_id "JLCImport:CL05B104KB54PNC")
+		(at 20.32 40.64 90)
+		(unit 1)
+		(body_style 1)
+		(exclude_from_sim no)
+		(in_bom yes)
+		(on_board yes)
+		(in_pos_files yes)
+		(dnp no)
+		(property "Reference" "C108"
+			(at 15.24 39.624 90)
+			(show_name no)
+			(do_not_autoplace no)
+			(effects
+				(font
+					(size 1.27 1.27)
+				)
+			)
+		)
+		(property "Value" "100nF 50V"
+			(at 19.05 37.592 90)
+			(show_name no)
+			(do_not_autoplace no)
+			(effects
+				(font
+					(size 1.27 1.27)
+				)
+			)
+		)
+		(property "Footprint" "Capacitor_SMD:C_0402_1005Metric"
+			(at 20.32 40.64 0)
+			(hide yes)
+			(show_name no)
+			(do_not_autoplace no)
+			(effects
+				(font
+					(size 1.27 1.27)
+				)
+			)
+		)
+		(property "Datasheet" "https://www.lcsc.com/datasheet/lcsc_datasheet_2304140030_Samsung-Electro-Mechanics-CL05B104KB54PNC_C307331.pdf"
+			(at 20.32 40.64 0)
+			(hide yes)
+			(show_name no)
+			(do_not_autoplace no)
+			(effects
+				(font
+					(size 1.27 1.27)
+				)
+			)
+		)
+		(property "Description" "100nF 50V X7R ±10% 0402 Multilayer Ceramic Capacitors MLCC - SMD/SMT ROHS"
+			(at 20.32 40.64 0)
+			(hide yes)
+			(show_name no)
+			(do_not_autoplace no)
+			(effects
+				(font
+					(size 1.27 1.27)
+				)
+			)
+		)
+		(property "LCSC" "C307331"
+			(at 20.32 40.64 0)
+			(hide yes)
+			(show_name no)
+			(do_not_autoplace no)
+			(effects
+				(font
+					(size 1.27 1.27)
+				)
+			)
+		)
+		(property "Manufacturer" "Samsung Electro-Mechanics"
+			(at 20.32 40.64 0)
+			(hide yes)
+			(show_name no)
+			(do_not_autoplace no)
+			(effects
+				(font
+					(size 1.27 1.27)
+				)
+			)
+		)
+		(property "Manufacturer Part" "CL05B104KB54PNC"
+			(at 20.32 40.64 0)
+			(hide yes)
+			(show_name no)
+			(do_not_autoplace no)
+			(effects
+				(font
+					(size 1.27 1.27)
+				)
+			)
+		)
+		(pin "2"
+		)
+		(pin "1"
+		)
+		(instances
+			(project "DrunkEarPhoneAdapter"
+				(path "/df940915-8af0-46f9-b18a-23d4684ae671/c6b936ac-23e1-4f20-8d3d-ded05833abcb"
+					(reference "C108")
+					(unit 1)
+				)
